Commit message: fix: simulator fixed

File: lv2_module6/urdf/beebot.urdf.xacro (robot description, xacro)
@@ -153,4 +153,49 @@
   </joint>
   <!-- ================= 선가이드 폴 (뒤쪽 끝) + pole_cam ================= -->
+  <!-- 적재함 (뒤쪽 절반, 퍽 운반): 바닥 윗면 z=0.140 (base_link 기준) · 가이드벽 4면 (높이 0.04, 두께 0.005)
+       시뮬레이터는 같은 치수로 퍽 받침·가둠 판정 (simulator/main.py TRAY) -->
+  <xacro:property name="tray_x0" value="-0.19"/>
+  <xacro:property name="tray_x1" value="-0.07"/>
+  <xacro:property name="tray_y" value="0.10"/>
+  <xacro:property name="tray_floor_z" value="0.140"/>
+  <xacro:property name="tray_wall_h" value="0.04"/>
+  <xacro:property name="tray_wall_t" value="0.005"/>
+  <link name="tray_link">
+    <visual>
+      <origin xyz="-0.13 0 0.1375"/>
+      <geometry><box size="0.12 0.20 0.005"/></geometry>
+      <material name="grey"/>
+    </visual>
+    <visual>
+      <origin xyz="-0.1875 0 0.16"/>
+      <geometry><box size="0.005 0.20 0.04"/></geometry>
+      <material name="grey"/>
+    </visual>
+    <visual>
+      <origin xyz="-0.0725 0 0.16"/>
+      <geometry><box size="0.005 0.20 0.04"/></geometry>
+      <material name="grey"/>
+    </visual>
+    <visual>
+      <origin xyz="-0.13 0.0975 0.16"/>
+      <geometry><box size="0.11 0.005 0.04"/></geometry>
+      <material name="grey"/>
+    </visual>
+    <visual>
+      <origin xyz="-0.13 -0.0975 0.16"/>
+      <geometry><box size="0.11 0.005 0.04"/></geometry>
+      <material name="grey"/>
+    </visual>
+    <collision>
+      <origin xyz="-0.13 0 0.1375"/>
+      <geometry><box size="0.12 0.20 0.005"/></geometry>
+    </collision>
+    <xacro:box_inertia m="0.05" x="0.12" y="0.20" z="0.005"><origin xyz="-0.13 0 0.1375"/></xacro:box_inertia>
+  </link>
+  <joint name="tray_joint" type="fixed">
+    <parent link="base_link"/>
+    <child link="tray_link"/>
+    <origin xyz="0 0 0"/>
+  </joint>
   <link name="cable_pole_link">
     <visual>

Commit message: feature: urdf update

File: lv2_module6/urdf/beebot.urdf.xacro (robot description, xacro)
@@ -1,20 +1,16 @@
 <?xml version="1.0"?>
 <!--
-  beebot — TurtleBot3 Waffle Pi + 앞쪽 상판(한 단) 위 매니퓰레이터(OM-X + 손목 roll + 그리퍼) + 뒤쪽 전원선 가이드 폴 (더미 치수)
+  beebot — 실측 CAD(bee.urdf, SolidWorks 내보내기)에서 만든 모델. bee.urdf를 새로 받으면 이 파일을 다시 만든다:
+    · 메시 경로: meshes/x.stl → package://ros_system/urdf/meshes/x.stl
+    · 이름 맞춤(제어·시뮬레이터가 쓰는 이름): camera_rear → pole_cam, camera_wrist → gripper_cam,
+      gripper_joint → gripper_left_joint, gripper_mimic_joint → gripper_right_joint, tcp → end_effector
+    · 추가: imu_link · <ros2_control> 블록(BeebotSystemHardware) · xacro 인자
   설계: documents/ros2-design/07-tf.md (TF 트리), 08-ctrl.md (ros2_control)
   좌표: base_footprint(바닥) → base_link(바퀴 축 아래 0.010m), x 앞 · y 왼쪽 · z 위
-    - 차체: Waffle Pi 본체 266×266mm, 바퀴 반경 0.033m · 간격 0.287m, 뒤쪽 캐스터 2개
-    - 상판(deck): 차체 위 앞쪽 절반만 덮는 판넬, 스탠드오프 0.05m 위
-    - 매니퓰레이터: 상판 위 OpenMANIPULATOR-X + 손목 roll — 구동 관절 6개
-        joint1 yaw · joint2~4 pitch (OM-X) · joint5 손목 roll (추가) · gripper_left_joint (평행 그리퍼)
-    - 선가이드 폴: 차체 위 뒤쪽 끝, 전원선이 위에서 내려온다. pole_cam은 이 폴 위에 전방 하향으로 단다 (가정)
-    - gripper_cam: 그리퍼 몸체(gripper_link) 위에 얹은 RealSense
+  구동 관절 6개: joint1~5 (팔) · gripper_left_joint (평행 그리퍼, 0=닫힘 · 0.0265=열림, 오른쪽은 mimic) + 바퀴 2개
   xacro 인자:
     mock_hardware (false)  true면 control/BeebotSystemHardware가 실기 대신 명령을 그대로 상태로 되돌려 줌 (테스트베드)
     mock_effort   (0.0)    mock일 때 팔 관절 effort[A] (arm_safety_monitor 시험용)
     port          (/dev/ttyACM0)  OpenCR 포트
-  TODO(권형중): 실측 치수·질량, 메시 (OM-X는 ROBOTIS open_manipulator_description/meshes STL을 쓸 수 있음), 손목 roll 모듈 실제 길이
-  Isaac Sim용 USD는 이 파일을 xacro로 펼친 URDF를 Isaac Sim URDF Importer로 변환해 만든다:
-    xacro beebot.urdf.xacro > beebot.urdf
 -->
 <robot name="beebot" xmlns:xacro="http://www.ros.org/wiki/xacro">
@@ -22,302 +18,384 @@
   <xacro:arg name="mock_effort" default="0.0"/>
   <xacro:arg name="port" default="/dev/ttyACM0"/>
-  <xacro:property name="PI" value="3.14159265"/>
-  <!-- 차체 -->
-  <xacro:property name="wheel_radius" value="0.033"/>
-  <xacro:property name="wheel_width" value="0.018"/>
-  <xacro:property name="wheel_separation" value="0.287"/>
-  <xacro:property name="body_l" value="0.266"/>
-  <xacro:property name="body_w" value="0.266"/>
-  <xacro:property name="body_h" value="0.110"/>
-  <xacro:property name="body_x" value="-0.064"/>   <!-- 바퀴 축 기준 본체 중심 (바퀴가 앞쪽) -->
-  <xacro:property name="body_z" value="0.080"/>
-  <xacro:property name="body_top" value="${body_z + body_h / 2}"/>
-  <!-- 상판: 본체 앞쪽 절반 -->
-  <xacro:property name="deck_standoff" value="0.050"/>
-  <xacro:property name="deck_t" value="0.005"/>
-  <xacro:property name="deck_l" value="${body_l / 2}"/>
-  <xacro:property name="deck_x" value="${body_x + body_l / 4}"/>
-  <xacro:property name="deck_top" value="${body_top + deck_standoff + deck_t}"/>
-  <!-- 선가이드 폴: 본체 뒤쪽 끝 -->
-  <xacro:property name="pole_h" value="0.450"/>
-  <xacro:property name="pole_r" value="0.010"/>
-  <xacro:property name="pole_x" value="${body_x - body_l / 2 + 0.020}"/>
-  <material name="dark"><color rgba="0.2 0.2 0.2 1"/></material>
-  <material name="grey"><color rgba="0.6 0.6 0.6 1"/></material>
-  <material name="white"><color rgba="0.95 0.95 0.95 1"/></material>
-  <material name="orange"><color rgba="0.95 0.5 0.1 1"/></material>
-  <material name="blue"><color rgba="0.2 0.4 0.8 1"/></material>
-  <!-- 관성: 균질 직육면체·원기둥·구 -->
-  <xacro:macro name="box_inertia" params="m x y z *origin">
-    <inertial>
-      <xacro:insert_block name="origin"/>
-      <mass value="${m}"/>
-      <inertia ixx="${m * (y*y + z*z) / 12}" ixy="0" ixz="0" iyy="${m * (x*x + z*z) / 12}" iyz="0" izz="${m * (x*x + y*y) / 12}"/>
-    </inertial>
-  </xacro:macro>
-  <xacro:macro name="cylinder_inertia" params="m r h *origin">
-    <inertial>
-      <xacro:insert_block name="origin"/>
-      <mass value="${m}"/>
-      <inertia ixx="${m * (3*r*r + h*h) / 12}" ixy="0" ixz="0" iyy="${m * (3*r*r + h*h) / 12}" iyz="0" izz="${m * r * r / 2}"/>
-    </inertial>
-  </xacro:macro>
-  <!-- ================= 베이스 ================= -->
   <link name="base_footprint"/>
-  <link name="base_link">
-    <visual>
-      <origin xyz="${body_x} 0 ${body_z}"/>
-      <geometry><box size="${body_l} ${body_w} ${body_h}"/></geometry>
-      <material name="dark"/>
-    </visual>
-    <collision>
-      <origin xyz="${body_x} 0 ${body_z}"/>
-      <geometry><box size="${body_l} ${body_w} ${body_h}"/></geometry>
-    </collision>
-    <xacro:box_inertia m="1.5" x="${body_l}" y="${body_w}" z="${body_h}"><origin xyz="${body_x} 0 ${body_z}"/></xacro:box_inertia>
-  </link>
   <joint name="base_joint" type="fixed">
     <parent link="base_footprint"/>
     <child link="base_link"/>
-    <origin xyz="0 0 0.010"/>
-  </joint>
-  <xacro:macro name="wheel" params="side y">
-    <link name="wheel_${side}_link">
-      <visual>
-        <origin rpy="${-PI/2} 0 0"/>
-        <geometry><cylinder radius="${wheel_radius}" length="${wheel_width}"/></geometry>
-        <material name="grey"/>
-      </visual>
-      <collision>
-        <origin rpy="${-PI/2} 0 0"/>
-        <geometry><cylinder radius="${wheel_radius}" length="${wheel_width}"/></geometry>
-      </collision>
-      <xacro:cylinder_inertia m="0.03" r="${wheel_radius}" h="${wheel_width}"><origin rpy="${-PI/2} 0 0"/></xacro:cylinder_inertia>
-    </link>
-    <joint name="wheel_${side}_joint" type="continuous">
-      <parent link="base_link"/>
-      <child link="wheel_${side}_link"/>
-      <origin xyz="0 ${y} ${wheel_radius - 0.010}"/>
-      <axis xyz="0 1 0"/>
-    </joint>
-  </xacro:macro>
-  <xacro:wheel side="left" y="${wheel_separation / 2}"/>
-  <xacro:wheel side="right" y="${-wheel_separation / 2}"/>
-  <xacro:macro name="caster" params="side y">
-    <link name="caster_${side}_link">
-      <collision><geometry><sphere radius="0.010"/></geometry></collision>
-      <inertial><mass value="0.005"/><inertia ixx="1e-7" ixy="0" ixz="0" iyy="1e-7" iyz="0" izz="1e-7"/></inertial>
-    </link>
-    <joint name="caster_${side}_joint" type="fixed">
-      <parent link="base_link"/>
-      <child link="caster_${side}_link"/>
-      <origin xyz="${body_x - body_l / 2 + 0.020} ${y} 0.000"/>
-    </joint>
-  </xacro:macro>
-  <xacro:caster side="left" y="0.064"/>
-  <xacro:caster side="right" y="-0.064"/>
+    <origin rpy="0.000000 -0.000000 0.000000" xyz="0.000000 0.000000 0.010000"/>
+  </joint>
+  <link name="base_link">
+    <inertial>
+      <origin rpy="0 0 0" xyz="-0.085631 -0.000202 0.080552"/>
+      <mass value="2.400600"/>
+      <inertia ixx="2.8115e-02" ixy="-1.1729e-05" ixz="6.3963e-03" iyy="3.2571e-02" iyz="-7.6014e-06" izz="2.7719e-02"/>
+    </inertial>
+    <visual>
+      <origin rpy="0 0 0" xyz="0 0 0"/>
+      <geometry>
+        <mesh filename="package://ros_system/urdf/meshes/base_link.stl" scale="0.001 0.001 0.001"/>
+      </geometry>
+    </visual>
+    <collision>
+      <origin rpy="0.000000 0.000000 0.000000" xyz="-0.081850 0.000000 0.063175"/>
+      <geometry>
+        <box size="0.301300 0.265600 0.126350"/>
+      </geometry>
+    </collision>
+    <collision>
+      <origin rpy="0.000000 0.000000 0.000000" xyz="0.032000 0.000000 0.131250"/>
+      <geometry>
+        <box size="0.073600 0.137600 0.009800"/>
+      </geometry>
+    </collision>
+    <collision>
+      <origin rpy="0.000000 0.000000 0.000000" xyz="-0.209400 0.000000 0.291900"/>
+      <geometry>
+        <box size="0.020000 0.020000 0.331100"/>
+      </geometry>
+    </collision>
+    <collision>
+      <origin rpy="0 0 0" xyz="-0.177000 0.064000 -0.005237"/>
+      <geometry>
+        <sphere radius="0.004763"/>
+      </geometry>
+    </collision>
+    <collision>
+      <origin rpy="0 0 0" xyz="-0.177000 -0.064000 -0.005237"/>
+      <geometry>
+        <sphere radius="0.004763"/>
+      </geometry>
+    </collision>
+  </link>
+  <joint name="wheel_left_joint" type="continuous">
+    <parent link="base_link"/>
+    <child link="wheel_left_link"/>
+    <origin rpy="0.000000 -0.000000 0.000000" xyz="0.000000 0.143900 0.023000"/>
+    <axis xyz="0 1 0"/>
+    <limit effort="3.0" velocity="8.063"/>
+  </joint>
+  <link name="wheel_left_link">
+    <inertial>
+      <origin rpy="0 0 0" xyz="0.000000 -0.000704 0.000002"/>
+      <mass value="0.028500"/>
+      <inertia ixx="1.1098e-05" ixy="5.7318e-09" ixz="3.1818e-09" iyy="2.0549e-05" iyz="-4.8114e-11" izz="1.1095e-05"/>
+    </inertial>
+    <visual>
+      <origin rpy="0 0 0" xyz="0 0 0"/>
+      <geometry>
+        <mesh filename="package://ros_system/urdf/meshes/wheel_left_link.stl" scale="0.001 0.001 0.001"/>
+      </geometry>
+    </visual>
+    <collision>
+      <origin rpy="1.570796 0 0" xyz="0 0 0"/>
+      <geometry>
+        <cylinder length="0.018200" radius="0.033000"/>
+      </geometry>
+    </collision>
+  </link>
+  <joint name="wheel_right_joint" type="continuous">
+    <parent link="base_link"/>
+    <child link="wheel_right_link"/>
+    <origin rpy="0.000000 -0.000000 0.000000" xyz="0.000000 -0.143900 0.023000"/>
+    <axis xyz="0 1 0"/>
+    <limit effort="3.0" velocity="8.063"/>
+  </joint>
+  <link name="wheel_right_link">
+    <inertial>
+      <origin rpy="0 0 0" xyz="0.000000 0.000704 -0.000002"/>
+      <mass value="0.028500"/>
+      <inertia ixx="1.1098e-05" ixy="-5.7318e-09" ixz="-3.1818e-09" iyy="2.0549e-05" iyz="-4.8114e-11" izz="1.1095e-05"/>
+    </inertial>
+    <visual>
+      <origin rpy="0 0 0" xyz="0 0 0"/>
+      <geometry>
+        <mesh filename="package://ros_system/urdf/meshes/wheel_right_link.stl" scale="0.001 0.001 0.001"/>
+      </geometry>
+    </visual>
+    <collision>
+      <origin rpy="1.570796 0 0" xyz="0 0 0"/>
+      <geometry>
+        <cylinder length="0.018200" radius="0.033000"/>
+      </geometry>
+    </collision>
+  </link>
+  <joint name="pole_cam_joint" type="fixed">
+    <parent link="base_link"/>
+    <child link="pole_cam_link"/>
+    <origin rpy="0.000000 0.314159 0.000000" xyz="-0.137869 0.000185 0.417108"/>
+  </joint>
+  <link name="pole_cam_link">
+    <inertial>
+      <origin rpy="0 0 0" xyz="-0.013393 0.001408 -0.000023"/>
+      <mass value="0.072000"/>
+      <inertia ixx="4.6203e-05" ixy="4.1597e-07" ixz="2.0009e-08" iyy="6.9218e-06" iyz="3.6648e-09" izz="4.6614e-05"/>
+    </inertial>
+    <visual>
+      <origin rpy="0 0 0" xyz="0 0 0"/>
+      <geometry>
+        <mesh filename="package://ros_system/urdf/meshes/camera_rear_link.stl" scale="0.001 0.001 0.001"/>
+      </geometry>
+    </visual>
+    <collision>
+      <origin rpy="0.000000 0.000000 0.000000" xyz="-0.012525 -0.000058 -0.000000"/>
+      <geometry>
+        <box size="0.025050 0.089714 0.025000"/>
+      </geometry>
+    </collision>
+  </link>
+  <joint name="arm_mount_joint" type="fixed">
+    <parent link="base_link"/>
+    <child link="arm_base_link"/>
+    <origin rpy="-0.000000 0.000000 0.000000" xyz="0.051045 -0.000000 0.134795"/>
+  </joint>
+  <link name="arm_base_link">
+    <inertial>
+      <origin rpy="0.0 0.0 0.0" xyz="-0.01169226743052282 -3.774353380840405e-15 0.023926534323405226"/>
+      <mass value="0.08108257974970318"/>
+      <inertia ixx="1.2862502962900217e-05" ixy="6.251056457349735e-19" ixz="-1.811662342359175e-07" iyy="2.2531969968508323e-05" iyz="1.5086560978736273e-17" izz="1.9821050957242446e-05"/>
+    </inertial>
+    <visual name="arm_base_link_visual">
+      <origin rpy="0.0 -0.0 0.0" xyz="0.0 0.0 0.0"/>
+      <geometry>
+        <mesh filename="package://ros_system/urdf/meshes/arm_base_1.stl" scale="0.001 0.001 0.001"/>
+      </geometry>
+    </visual>
+    <collision name="arm_base_link_collision">
+      <origin rpy="0.0 -0.0 0.0" xyz="0.0 0.0 0.0"/>
+      <geometry>
+        <mesh filename="package://ros_system/urdf/meshes/arm_base_1.stl" scale="0.001 0.001 0.001"/>
+      </geometry>
+    </collision>
+  </link>
+  <link name="shoulder_link">
+    <inertial>
+      <origin rpy="0.0 -0.0 0.0" xyz="1.3576596988624524e-13 0.0006685783443131954 0.028869490461060965"/>
+      <mass value="0.08583374201044289"/>
+      <inertia ixx="2.6324742259425243e-05" ixy="-7.312006911381859e-16" ixz="-9.128905585988183e-18" iyy="2.2861624315008813e-05" iyz="-8.980408739570743e-08" izz="1.4187591495603722e-05"/>
+    </inertial>
+    <visual name="shoulder_link_visual">
+      <origin rpy="-2.220438457117713e-16 -0.0 0.0" xyz="2.493290125897981e-18 -9.081593289611446e-18 -0.0409"/>
+      <geometry>
+        <mesh filename="package://ros_system/urdf/meshes/shoulder_1.stl" scale="0.001 0.001 0.001"/>
+      </geometry>
+    </visual>
+    <collision name="shoulder_link_collision">
+      <origin rpy="-2.220438457117713e-16 -0.0 0.0" xyz="2.493290125897981e-18 -9.081593289611446e-18 -0.0409"/>
+      <geometry>
+        <mesh filename="package://ros_system/urdf/meshes/shoulder_1.stl" scale="0.001 0.001 0.001"/>
+      </geometry>
+    </collision>
+  </link>
+  <link name="upper_arm_link">
+    <inertial>
+      <origin rpy="0.0 -3.1860094989889126e-35 0.0" xyz="-0.008487065074045876 0.10499673065502067 0.019195324443247258"/>
+      <mass value="0.12886465633856012"/>
+      <inertia ixx="0.00018774476358412258" ixy="2.3927185167595554e-05" ixz="2.494779573069466e-07" iyy="3.578068745086586e-05" iyz="-1.3200789827030247e-06" izz="0.00019584173585813564"/>
+    </inertial>
+    <visual name="upper_arm_link_visual">
+      <origin rpy="1.570796326794511 -2.1442092918336785e-10 3.141592653589793" xyz="4.0203924221813285e-12 -0.08250000000000723 0.0187499999999682"/>
+      <geometry>
+        <mesh filename="package://ros_system/urdf/meshes/link1_1.stl" scale="0.001 0.001 0.001"/>
+      </geometry>
+    </visual>
+    <collision name="upper_arm_link_collision">
+      <origin rpy="1.570796326794511 -2.1442092918336785e-10 3.141592653589793" xyz="4.0203924221813285e-12 -0.08250000000000723 0.0187499999999682"/>
+      <geometry>
+        <mesh filename="package://ros_system/urdf/meshes/link1_1.stl" scale="0.001 0.001 0.001"/>
+      </geometry>
+    </collision>
+  </link>
+  <link name="forearm_link">
+    <inertial>
+      <origin rpy="0.0 -4.32741592896883e-38 0.0" xyz="-0.09379595988179056 6.576999203034006e-07 0.019239230160790734"/>
+      <mass value="0.117299760592073"/>
+      <inertia ixx="1.9524545623177503e-05" ixy="-2.9158900918577e-09" ixz="1.0925502645848908e-06" iyy="0.00014316575812332259" iyz="3.773501040795638e-11" izz="0.00013706538722077516"/>
+    </inertial>
+    <visual name="forearm_link_visual">
+      <origin rpy="1.5707963267949108 -2.1428325780447923e-10 3.141592653589793" xyz="0.02400000000401781 -0.21049999999999977 0.018749999994860194"/>
+      <geometry>
+        <mesh filename="package://ros_system/urdf/meshes/link2_1.stl" scale="0.001 0.001 0.001"/>
+      </geometry>
+    </visual>
+    <collision name="forearm_link_collision">
+      <origin rpy="1.5707963267949108 -2.1428325780447923e-10 3.141592653589793" xyz="0.02400000000401781 -0.21049999999999977 0.018749999994860194"/>
+      <geometry>
+        <mesh filename="package://ros_system/urdf/meshes/link2_1.stl" scale="0.001 0.001 0.001"/>
+      </geometry>
+    </collision>
+  </link>
+  <link name="wrist_link">
+    <inertial>
+      <origin rpy="0.0 -2.4338940029490826e-38 0.0" xyz="-0.04362261924950845 0.011448916236659308 0.018749999965138587"/>
+      <mass value="0.09015230299876778"/>
+      <inertia ixx="2.376831067770098e-05" ixy="5.954218246732174e-07" ixz="-3.5110061152839838e-15" iyy="1.98868978503507e-05" iyz="2.3069523907684884e-16" izz="2.9205178935103743e-05"/>
+    </inertial>
+    <visual name="wrist_link_visual">
+      <origin rpy="1.570796326794886 -2.14258832897939e-10 3.141592653589793" xyz="0.14800000000401736 -0.21050000000000021 0.01874999996828745"/>
+      <geometry>
+        <mesh filename="package://ros_system/urdf/meshes/wrist_1.stl" scale="0.001 0.001 0.001"/>
+      </geometry>
+    </visual>
+    <collision name="wrist_link_collision">
+      <origin rpy="1.570796326794886 -2.14258832897939e-10 3.141592653589793" xyz="0.14800000000401736 -0.21050000000000021 0.01874999996828745"/>
+      <geometry>
+        <mesh filename="package://ros_system/urdf/meshes/wrist_1.stl" scale="0.001 0.001 0.001"/>
+      </geometry>
+    </collision>
+  </link>
+  <link name="gripper_link">
+    <inertial>
+      <origin rpy="0.0 -0.0 0.0" xyz="-1.5886903241172202e-07 -0.008076961447025325 0.033331202092510386"/>
+      <mass value="0.17574131271191906"/>
+      <inertia ixx="7.566997046639816e-05" ixy="4.58037525130514e-08" ixz="1.147686837904163e-09" iyy="0.00010679192530828156" iyz="-8.666284099644634e-06" izz="0.00010974001130350429"/>
+    </inertial>
+    <visual name="gripper_link_visual">
+      <origin rpy="1.5707963267948966 -1.5707963265806377 0" xyz="4.518721444630066e-11 0.21050000000000002 -0.2109"/>
+      <geometry>
+        <mesh filename="package://ros_system/urdf/meshes/gripper_body_1.stl" scale="0.001 0.001 0.001"/>
+      </geometry>
+    </visual>
+    <collision name="gripper_link_collision">
+      <origin rpy="1.5707963267948966 -1.5707963265806377 0" xyz="4.518721444630066e-11 0.21050000000000002 -0.2109"/>
+      <geometry>
+        <mesh filename="package://ros_system/urdf/meshes/gripper_body_1.stl" scale="0.001 0.001 0.001"/>
+      </geometry>
+    </collision>
+  </link>
+  <link name="finger_left_link">
+    <inertial>
+      <origin rpy="0.0 -2.994698132526971e-39 0.0" xyz="-0.021558941309427697 -8.180647438322807e-06 0.018420805920369158"/>
+      <mass value="0.0535652061896923"/>
+      <inertia ixx="1.6044439735299576e-05" ixy="3.5963237118778324e-09" ixz="4.605246566927584e-06" iyy="3.0067540639167056e-05" iyz="1.5747727444362111e-09" izz="3.8262391196432324e-05"/>
+    </inertial>
+    <visual name="finger_left_link_visual">
+      <origin rpy="-1.5707963267949108 -1.4829026895313252e-11 3.141592653589793" xyz="0.2640500000005726 0.21049999999999947 0.03861386999608739"/>
+      <geometry>
+        <mesh filename="package://ros_system/urdf/meshes/finger_R_1.stl" scale="0.001 0.001 0.001"/>
+      </geometry>
+    </visual>
+    <collision name="finger_left_link_collision">
+      <origin rpy="-1.5707963267949108 -1.4829026895313252e-11 3.141592653589793" xyz="0.2640500000005726 0.21049999999999947 0.03861386999608739"/>
+      <geometry>
+        <mesh filename="package://ros_system/urdf/meshes/finger_R_1.stl" scale="0.001 0.001 0.001"/>
+      </geometry>
+    </collision>
+  </link>
+  <link name="finger_right_link">
+    <inertial>
+      <origin rpy="0.0 2.994698132526979e-39 0.0" xyz="-0.02155799088002368 -8.180633800094484e-06 0.01842080593956481"/>
+      <mass value="0.05356520623406594"/>
+      <inertia ixx="1.6044441819699544e-05" ixy="3.5958195413410427e-09" ixz="4.605674889789638e-06" iyy="3.0069181530455354e-05" iyz="1.5747659279198598e-09" izz="3.826403413411749e-05"/>
+    </inertial>
+    <visual name="finger_right_link_visual">
+      <origin rpy="1.5707963267948823 1.4829026895313265e-11 3.141592653589793" xyz="0.2640499999994274 -0.21050000000000055 0.038613870003912615"/>
+      <geometry>
+        <mesh filename="package://ros_system/urdf/meshes/finger_L_1.stl" scale="0.001 0.001 0.001"/>
+      </geometry>
+    </visual>
+    <collision name="finger_right_link_collision">
+      <origin rpy="1.5707963267948823 1.4829026895313265e-11 3.141592653589793" xyz="0.2640499999994274 -0.21050000000000055 0.038613870003912615"/>
+      <geometry>
+        <mesh filename="package://ros_system/urdf/meshes/finger_L_1.stl" scale="0.001 0.001 0.001"/>
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