Commit message: feat: add storage collision

File: lv2_module6/urdf/beebot.urdf.xacro (robot description, xacro)
@@ -1,6 +1,6 @@
-<?xml version="1.0"?>
+<?xml version="1.0" ?>
 <!--
   beebot — 실측 CAD(bee.urdf, SolidWorks 내보내기)에서 만든 모델. bee.urdf를 새로 받으면 이 파일을 다시 만든다:
-    · 메시 경로: meshes/x.stl → package://ros_system/urdf/meshes/x.stl
+    · 메시 경로: meshes/x.stl → meshes/x.stl
     · 이름 맞춤(제어·시뮬레이터가 쓰는 이름): camera_rear → pole_cam, camera_wrist → gripper_cam,
       gripper_joint → gripper_left_joint, gripper_mimic_joint → gripper_right_joint, tcp → end_effector
@@ -14,8 +14,10 @@
     port          (/dev/ttyACM0)  OpenCR 포트
 -->
+<!-- generated by make_xacro.py -->
 <robot name="beebot" xmlns:xacro="http://www.ros.org/wiki/xacro">
   <xacro:arg name="mock_hardware" default="false"/>
   <xacro:arg name="mock_effort" default="0.0"/>
   <xacro:arg name="port" default="/dev/ttyACM0"/>
+  <xacro:arg name="mesh_uri" default="package://ros_system/urdf/meshes"/>
   <link name="base_footprint"/>
   <joint name="base_joint" type="fixed">
@@ -33,11 +35,23 @@
       <origin rpy="0 0 0" xyz="0 0 0"/>
       <geometry>
-        <mesh filename="package://ros_system/urdf/meshes/base_link.stl" scale="0.001 0.001 0.001"/>
-      </geometry>
-    </visual>
-    <collision>
-      <origin rpy="0.000000 0.000000 0.000000" xyz="-0.081850 0.000000 0.063175"/>
-      <geometry>
-        <box size="0.301300 0.265600 0.126350"/>
+        <mesh filename="$(arg mesh_uri)/base_link.stl" scale="0.001 0.001 0.001"/>
+      </geometry>
+    </visual>
+    <collision>
+      <origin rpy="0.000000 0.000000 0.000000" xyz="-0.081850 0.000000 0.045500"/>
+      <geometry>
+        <box size="0.301300 0.265600 0.091000"/>
+      </geometry>
+    </collision>
+    <collision>
+      <origin rpy="0.000000 0.000000 0.000000" xyz="0.032000 0.000000 0.108675"/>
+      <geometry>
+        <box size="0.073600 0.137600 0.035350"/>
+      </geometry>
+    </collision>
+    <collision>
+      <origin rpy="0.000000 0.000000 0.000000" xyz="-0.209400 0.000000 0.108675"/>
+      <geometry>
+        <box size="0.020000 0.020000 0.035350"/>
       </geometry>
     </collision>
@@ -64,4 +78,58 @@
       <geometry>
         <sphere radius="0.004763"/>
+      </geometry>
+    </collision>
+    <collision name="storage_collision_0">
+      <origin rpy="1.570796 0.000000 0.000000" xyz="-0.064000 0.000000 -0.000500"/>
+      <geometry>
+        <mesh filename="$(arg mesh_uri)/storage_collision/storage_0.stl" scale="0.001 0.001 0.001"/>
+      </geometry>
+    </collision>
+    <collision name="storage_collision_1">
+      <origin rpy="1.570796 0.000000 0.000000" xyz="-0.064000 0.000000 -0.000500"/>
+      <geometry>
+        <mesh filename="$(arg mesh_uri)/storage_collision/storage_1.stl" scale="0.001 0.001 0.001"/>
+      </geometry>
+    </collision>
+    <collision name="storage_collision_2">
+      <origin rpy="1.570796 0.000000 0.000000" xyz="-0.064000 0.000000 -0.000500"/>
+      <geometry>
+        <mesh filename="$(arg mesh_uri)/storage_collision/storage_2.stl" scale="0.001 0.001 0.001"/>
+      </geometry>
+    </collision>
+    <collision name="storage_collision_3">
+      <origin rpy="1.570796 0.000000 0.000000" xyz="-0.064000 0.000000 -0.000500"/>
+      <geometry>
+        <mesh filename="$(arg mesh_uri)/storage_collision/storage_3.stl" scale="0.001 0.001 0.001"/>
+      </geometry>
+    </collision>
+    <collision name="storage_collision_4">
+      <origin rpy="1.570796 0.000000 0.000000" xyz="-0.064000 0.000000 -0.000500"/>
+      <geometry>
+        <mesh filename="$(arg mesh_uri)/storage_collision/storage_4.stl" scale="0.001 0.001 0.001"/>
+      </geometry>
+    </collision>
+    <collision name="storage_collision_5">
+      <origin rpy="1.570796 0.000000 0.000000" xyz="-0.064000 0.000000 -0.000500"/>
+      <geometry>
+        <mesh filename="$(arg mesh_uri)/storage_collision/storage_5.stl" scale="0.001 0.001 0.001"/>
+      </geometry>
+    </collision>
+    <collision name="storage_collision_6">
+      <origin rpy="1.570796 0.000000 0.000000" xyz="-0.064000 0.000000 -0.000500"/>
+      <geometry>
+        <mesh filename="$(arg mesh_uri)/storage_collision/storage_6.stl" scale="0.001 0.001 0.001"/>
+      </geometry>
+    </collision>
+    <collision name="storage_collision_7">
+      <origin rpy="1.570796 0.000000 0.000000" xyz="-0.064000 0.000000 -0.000500"/>
+      <geometry>
+        <mesh filename="$(arg mesh_uri)/storage_collision/storage_7.stl" scale="0.001 0.001 0.001"/>
+      </geometry>
+    </collision>
+    <collision name="storage_collision_8">
+      <origin rpy="1.570796 0.000000 0.000000" xyz="-0.064000 0.000000 -0.000500"/>
+      <geometry>
+        <mesh filename="$(arg mesh_uri)/storage_collision/storage_8.stl" scale="0.001 0.001 0.001"/>
       </geometry>
     </collision>
@@ -83,5 +151,5 @@
       <origin rpy="0 0 0" xyz="0 0 0"/>
       <geometry>
-        <mesh filename="package://ros_system/urdf/meshes/wheel_left_link.stl" scale="0.001 0.001 0.001"/>
+        <mesh filename="$(arg mesh_uri)/wheel_left_link.stl" scale="0.001 0.001 0.001"/>
       </geometry>
     </visual>
@@ -109,5 +177,5 @@
       <origin rpy="0 0 0" xyz="0 0 0"/>
       <geometry>
-        <mesh filename="package://ros_system/urdf/meshes/wheel_right_link.stl" scale="0.001 0.001 0.001"/>
+        <mesh filename="$(arg mesh_uri)/wheel_right_link.stl" scale="0.001 0.001 0.001"/>
       </geometry>
     </visual>
@@ -133,5 +201,5 @@
       <origin rpy="0 0 0" xyz="0 0 0"/>
       <geometry>
-        <mesh filename="package://ros_system/urdf/meshes/camera_rear_link.stl" scale="0.001 0.001 0.001"/>
+        <mesh filename="$(arg mesh_uri)/camera_rear_link.stl" scale="0.001 0.001 0.001"/>
       </geometry>
     </visual>
@@ -157,5 +225,5 @@
       <origin rpy="0.0 -0.0 0.0" xyz="0.0 0.0 0.0"/>
       <geometry>
-        <mesh filename="package://ros_system/urdf/meshes/arm_base_1.stl" scale="0.001 0.001 0.001"/>
+        <mesh filename="$(arg mesh_uri)/arm_base_1.stl" scale="0.001 0.001 0.001"/>
       </geometry>
     </visual>
@@ -163,5 +231,5 @@
       <origin rpy="0.0 -0.0 0.0" xyz="0.0 0.0 0.0"/>
       <geometry>
-        <mesh filename="package://ros_system/urdf/meshes/arm_base_1.stl" scale="0.001 0.001 0.001"/>
+        <mesh filename="$(arg mesh_uri)/arm_base_1.stl" scale="0.001 0.001 0.001"/>
       </geometry>
     </collision>
@@ -176,5 +244,5 @@
       <origin rpy="-2.220438457117713e-16 -0.0 0.0" xyz="2.493290125897981e-18 -9.081593289611446e-18 -0.0409"/>
       <geometry>
-        <mesh filename="package://ros_system/urdf/meshes/shoulder_1.stl" scale="0.001 0.001 0.001"/>
+        <mesh filename="$(arg mesh_uri)/shoulder_1.stl" scale="0.001 0.001 0.001"/>
       </geometry>
     </visual>
@@ -182,5 +250,5 @@
       <origin rpy="-2.220438457117713e-16 -0.0 0.0" xyz="2.493290125897981e-18 -9.081593289611446e-18 -0.0409"/>
       <geometry>
-        <mesh filename="package://ros_system/urdf/meshes/shoulder_1.stl" scale="0.001 0.001 0.001"/>
+        <mesh filename="$(arg mesh_uri)/shoulder_1.stl" scale="0.001 0.001 0.001"/>
       </geometry>
     </collision>
@@ -195,5 +263,5 @@
       <origin rpy="1.570796326794511 -2.1442092918336785e-10 3.141592653589793" xyz="4.0203924221813285e-12 -0.08250000000000723 0.0187499999999682"/>
       <geometry>
-        <mesh filename="package://ros_system/urdf/meshes/link1_1.stl" scale="0.001 0.001 0.001"/>
+        <mesh filename="$(arg mesh_uri)/link1_1.stl" scale="0.001 0.001 0.001"/>
       </geometry>
     </visual>
@@ -201,5 +269,5 @@
       <origin rpy="1.570796326794511 -2.1442092918336785e-10 3.141592653589793" xyz="4.0203924221813285e-12 -0.08250000000000723 0.0187499999999682"/>
       <geometry>
-        <mesh filename="package://ros_system/urdf/meshes/link1_1.stl" scale="0.001 0.001 0.001"/>
+        <mesh filename="$(arg mesh_uri)/link1_1.stl" scale="0.001 0.001 0.001"/>
       </geometry>
     </collision>
@@ -214,5 +282,5 @@
       <origin rpy="1.5707963267949108 -2.1428325780447923e-10 3.141592653589793" xyz="0.02400000000401781 -0.21049999999999977 0.018749999994860194"/>
       <geometry>
-        <mesh filename="package://ros_system/urdf/meshes/link2_1.stl" scale="0.001 0.001 0.001"/>
+        <mesh filename="$(arg mesh_uri)/link2_1.stl" scale="0.001 0.001 0.001"/>
       </geometry>
     </visual>
@@ -220,5 +288,5 @@
       <origin rpy="1.5707963267949108 -2.1428325780447923e-10 3.141592653589793" xyz="0.02400000000401781 -0.21049999999999977 0.018749999994860194"/>
       <geometry>
-        <mesh filename="package://ros_system/urdf/meshes/link2_1.stl" scale="0.001 0.001 0.001"/>
+        <mesh filename="$(arg mesh_uri)/link2_1.stl" scale="0.001 0.001 0.001"/>
       </geometry>
     </collision>
@@ -233,5 +301,5 @@
       <origin rpy="1.570796326794886 -2.14258832897939e-10 3.141592653589793" xyz="0.14800000000401736 -0.21050000000000021 0.01874999996828745"/>
       <geometry>
-        <mesh filename="package://ros_system/urdf/meshes/wrist_1.stl" scale="0.001 0.001 0.001"/>
+        <mesh filename="$(arg mesh_uri)/wrist_1.stl" scale="0.001 0.001 0.001"/>
       </geometry>
     </visual>
@@ -239,5 +307,5 @@
       <origin rpy="1.570796326794886 -2.14258832897939e-10 3.141592653589793" xyz="0.14800000000401736 -0.21050000000000021 0.01874999996828745"/>
       <geometry>
-        <mesh filename="package://ros_system/urdf/meshes/wrist_1.stl" scale="0.001 0.001 0.001"/>
+        <mesh filename="$(arg mesh_uri)/wrist_1.stl" scale="0.001 0.001 0.001"/>
       </geometry>
     </collision>
@@ -252,5 +320,5 @@
       <origin rpy="1.5707963267948966 -1.5707963265806377 0" xyz="4.518721444630066e-11 0.21050000000000002 -0.2109"/>
       <geometry>
-        <mesh filename="package://ros_system/urdf/meshes/gripper_body_1.stl" scale="0.001 0.001 0.001"/>
+        <mesh filename="$(arg mesh_uri)/gripper_body_1.stl" scale="0.001 0.001 0.001"/>
       </geometry>
     </visual>
@@ -258,5 +326,5 @@
       <origin rpy="1.5707963267948966 -1.5707963265806377 0" xyz="4.518721444630066e-11 0.21050000000000002 -0.2109"/>
       <geometry>
-        <mesh filename="package://ros_system/urdf/meshes/gripper_body_1.stl" scale="0.001 0.001 0.001"/>
+        <mesh filename="$(arg mesh_uri)/gripper_body_1.stl" scale="0.001 0.001 0.001"/>
       </geometry>
     </collision>
@@ -271,5 +339,5 @@
       <origin rpy="-1.5707963267949108 -1.4829026895313252e-11 3.141592653589793" xyz="0.2640500000005726 0.21049999999999947 0.03861386999608739"/>
       <geometry>
-        <mesh filename="package://ros_system/urdf/meshes/finger_R_1.stl" scale="0.001 0.001 0.001"/>
+        <mesh filename="$(arg mesh_uri)/finger_R_1.stl" scale="0.001 0.001 0.001"/>
       </geometry>
     </visual>
@@ -277,5 +345,5 @@
       <origin rpy="-1.5707963267949108 -1.4829026895313252e-11 3.141592653589793" xyz="0.2640500000005726 0.21049999999999947 0.03861386999608739"/>
       <geometry>
-        <mesh filename="package://ros_system/urdf/meshes/finger_R_1.stl" scale="0.001 0.001 0.001"/>
+        <mesh filename="$(arg mesh_uri)/finger_R_1.stl" scale="0.001 0.001 0.001"/>
       </geometry>
     </collision>
@@ -290,5 +358,5 @@
       <origin rpy="1.5707963267948823 1.4829026895313265e-11 3.141592653589793" xyz="0.2640499999994274 -0.21050000000000055 0.038613870003912615"/>
       <geometry>
-        <mesh filename="package://ros_system/urdf/meshes/finger_L_1.stl" scale="0.001 0.001 0.001"/>
+        <mesh filename="$(arg mesh_uri)/finger_L_1.stl" scale="0.001 0.001 0.001"/>
       </geometry>
     </visual>
@@ -296,5 +364,5 @@
       <origin rpy="1.5707963267948823 1.4829026895313265e-11 3.141592653589793" xyz="0.2640499999994274 -0.21050000000000055 0.038613870003912615"/>
       <geometry>
-        <mesh filename="package://ros_system/urdf/meshes/finger_L_1.stl" scale="0.001 0.001 0.001"/>
+        <mesh filename="$(arg mesh_uri)/finger_L_1.stl" scale="0.001 0.001 0.001"/>
       </geometry>
     </collision>
@@ -364,5 +432,5 @@
       <origin rpy="0 0 0" xyz="0 0 0"/>
       <geometry>
-        <mesh filename="package://ros_system/urdf/meshes/camera_wrist_link.stl" scale="0.001 0.001 0.001"/>
+        <mesh filename="$(arg mesh_uri)/camera_wrist_link.stl" scale="0.001 0.001 0.001"/>
       </geometry>
     </visual>
@@ -407,27 +475,51 @@
       <param name="baud_rate">1000000</param>
     </hardware>
-    <xacro:macro name="wheel_if" params="name">
-      <joint name="${name}">
-        <command_interface name="velocity"/>
-        <state_interface name="position"/>
-        <state_interface name="velocity"/>
-      </joint>
-    </xacro:macro>
-    <xacro:wheel_if name="wheel_left_joint"/>
-    <xacro:wheel_if name="wheel_right_joint"/>
-    <xacro:macro name="arm_if" params="name">
-      <joint name="${name}">
-        <command_interface name="position"/>
-        <state_interface name="position"/>
-        <state_interface name="velocity"/>
-        <state_interface name="effort"/>
-      </joint>
-    </xacro:macro>
-    <xacro:arm_if name="joint1"/>
-    <xacro:arm_if name="joint2"/>
-    <xacro:arm_if name="joint3"/>
-    <xacro:arm_if name="joint4"/>
-    <xacro:arm_if name="joint5"/>
-    <xacro:arm_if name="gripper_left_joint"/>   <!-- 오른쪽 손가락은 mimic (robot_state_publisher가 계산) -->
+    <joint name="wheel_left_joint">
+      <command_interface name="velocity"/>
+      <state_interface name="position"/>
+      <state_interface name="velocity"/>
+    </joint>
+    <joint name="wheel_right_joint">
+      <command_interface name="velocity"/>
+      <state_interface name="position"/>
+      <state_interface name="velocity"/>
+    </joint>
+    <joint name="joint1">
+      <command_interface name="position"/>
+      <state_interface name="position"/>
+      <state_interface name="velocity"/>
+      <state_interface name="effort"/>
+    </joint>
+    <joint name="joint2">
+      <command_interface name="position"/>
+      <state_interface name="position"/>
+      <state_interface name="velocity"/>
+      <state_interface name="effort"/>
+    </joint>
+    <joint name="joint3">
+      <command_interface name="position"/>
+      <state_interface name="position"/>
+      <state_interface name="velocity"/>
+      <state_interface name="effort"/>
+    </joint>
+    <joint name="joint4">
+      <command_interface name="position"/>
+      <state_interface name="position"/>
+      <state_interface name="velocity"/>
+      <state_interface name="effort"/>
+    </joint>
+    <joint name="joint5">
+      <command_interface name="position"/>
+      <state_interface name="position"/>
+      <state_interface name="velocity"/>
+      <state_interface name="effort"/>
+    </joint>
+    <joint name="gripper_left_joint">
+      <command_interface name="position"/>
+      <state_interface name="position"/>
+      <state_interface name="velocity"/>
+      <state_interface name="effort"/>
+    </joint>
+    <!-- 오른쪽 손가락은 mimic (robot_state_publisher가 계산) -->
     <sensor name="imu">
       <state_interface name="orientation.x"/>
