Commit message: feat: edit urdf

File: lv2_module6/urdf/beebot.urdf (robot description, URDF)
Before this commit: robot beebot, 18 links, 17 joints
Joints:
- joint arm_mount_joint: origin xyz=0.051045 -0.000000 0.134795 rpy=-0.000000 0.000000 0.000000 -> xyz=0.048019 0.000012 0.130149 rpy=-0.000000 0.000000 0.000000
- joint gripper_cam_joint: origin xyz=0.000504 -0.050245 0.080871 rpy=2.852763 -1.567096 -1.282111 -> xyz=0.000516 -0.054891 0.083897 rpy=2.852763 -1.567096 -1.282111

File: lv2_module6/urdf/beebot.urdf.xacro (robot description, xacro)
@@ -214,5 +214,5 @@
     <parent link="base_link"/>
     <child link="arm_base_link"/>
-    <origin rpy="-0.000000 0.000000 0.000000" xyz="0.051045 -0.000000 0.134795"/>
+    <origin rpy="-0.000000 0.000000 0.000000" xyz="0.048019 0.000012 0.130149"/>
   </joint>
   <link name="arm_base_link">
@@ -421,5 +421,5 @@
     <parent link="gripper_link"/>
     <child link="gripper_cam_link"/>
-    <origin rpy="2.852763 -1.567096 -1.282111" xyz="0.000504 -0.050245 0.080871"/>
+    <origin rpy="2.852763 -1.567096 -1.282111" xyz="0.000516 -0.054891 0.083897"/>
   </joint>
   <link name="gripper_cam_link">

Commit message: fix: wirst cam edit

File: lv2_module6/urdf/beebot.urdf (robot description, URDF)
Before this commit: robot beebot, 18 links, 17 joints
Links:
- added link basket_slot_0
- added link basket_slot_1
- added link basket_slot_10
- added link basket_slot_11
- added link basket_slot_2
- added link basket_slot_3
- added link basket_slot_4
- added link basket_slot_5
- added link basket_slot_6
- added link basket_slot_7
- added link basket_slot_8
- added link basket_slot_9
- link gripper_cam_link: geometry collision box size=0.055050 0.089714 0.045413; visual mesh filename=meshes/camera_wrist_link.stl scale=0.001 0.001 0.001
Joints:
- added joint basket_slot_0_joint: type fixed, parent base_link, child basket_slot_0, origin xyz=-0.16984 -0.0975 0.09125 rpy=0 0 0
- added joint basket_slot_10_joint: type fixed, parent base_link, child basket_slot_10, origin xyz=-0.03984 0.0325 0.09125 rpy=0 0 0
- added joint basket_slot_11_joint: type fixed, parent base_link, child basket_slot_11, origin xyz=-0.03984 0.0975 0.09125 rpy=0 0 0
- added joint basket_slot_1_joint: type fixed, parent base_link, child basket_slot_1, origin xyz=-0.16984 -0.0325 0.09125 rpy=0 0 0
- added joint basket_slot_2_joint: type fixed, parent base_link, child basket_slot_2, origin xyz=-0.16984 0.0325 0.09125 rpy=0 0 0
- added joint basket_slot_3_joint: type fixed, parent base_link, child basket_slot_3, origin xyz=-0.16984 0.0975 0.09125 rpy=0 0 0
- added joint basket_slot_4_joint: type fixed, parent base_link, child basket_slot_4, origin xyz=-0.10484 -0.0975 0.09125 rpy=0 0 0
- added joint basket_slot_5_joint: type fixed, parent base_link, child basket_slot_5, origin xyz=-0.10484 -0.0325 0.09125 rpy=0 0 0
- added joint basket_slot_6_joint: type fixed, parent base_link, child basket_slot_6, origin xyz=-0.10484 0.0325 0.09125 rpy=0 0 0
- added joint basket_slot_7_joint: type fixed, parent base_link, child basket_slot_7, origin xyz=-0.10484 0.0975 0.09125 rpy=0 0 0
- added joint basket_slot_8_joint: type fixed, parent base_link, child basket_slot_8, origin xyz=-0.03984 -0.0975 0.09125 rpy=0 0 0
- added joint basket_slot_9_joint: type fixed, parent base_link, child basket_slot_9, origin xyz=-0.03984 -0.0325 0.09125 rpy=0 0 0
- joint arm_mount_joint: origin xyz=0.048019 0.000012 0.130149 rpy=-0.000000 0.000000 0.000000 -> xyz=0.047985 -0.00023 0.130175 rpy=-0.000000 0.000000 0.000000
- joint gripper_cam_joint: origin xyz=0.000516 -0.054891 0.083897 rpy=2.852763 -1.567096 -1.282111 -> xyz=0.000273 -0.040325 0.081681 rpy=0.003448 -1.260182 1.567371
- joint gripper_cam_optical_joint: origin xyz=0.000000 0.000000 0.000000 rpy=-1.570796 0.000000 -1.570796 -> xyz=-0.004300 0.032500 0.000000 rpy=-1.570796 0.000000 -1.570796
- joint pole_cam_optical_joint: origin xyz=0.000000 0.000000 0.000000 rpy=-1.570796 0.000000 -1.570796 -> xyz=-0.004300 0.032500 0.000000 rpy=-1.570796 0.000000 -1.570796

File: lv2_module6/urdf/beebot.urdf.xacro (robot description, xacro)
@@ -214,5 +214,5 @@
     <parent link="base_link"/>
     <child link="arm_base_link"/>
-    <origin rpy="-0.000000 0.000000 0.000000" xyz="0.048019 0.000012 0.130149"/>
+    <origin rpy="-0.000000 0.000000 0.000000" xyz="0.047985 -0.00023 0.130175"/>
   </joint>
   <link name="arm_base_link">
@@ -421,11 +421,11 @@
     <parent link="gripper_link"/>
     <child link="gripper_cam_link"/>
-    <origin rpy="2.852763 -1.567096 -1.282111" xyz="0.000516 -0.054891 0.083897"/>
+    <origin rpy="0.003448 -1.260182 1.567371" xyz="0.000273 -0.040325 0.081681"/>
   </joint>
   <link name="gripper_cam_link">
     <inertial>
-      <origin rpy="0 0 0" xyz="-0.018065 0.001229 -0.001118"/>
+      <origin rpy="0 0 0" xyz="-0.017727 0.001229 -0.001059"/>
       <mass value="0.088370"/>
-      <inertia ixx="5.1972e-05" ixy="6.5780e-08" ixz="-2.7719e-06" iyy="1.8951e-05" iyz="-6.0902e-08" izz="6.0643e-05"/>
+      <inertia ixx="5.1824e-05" ixy="8.5769e-08" ixz="-2.1898e-06" iyy="1.7218e-05" iyz="-5.7372e-08" izz="5.9057e-05"/>
     </inertial>
     <visual>
@@ -436,7 +436,7 @@
     </visual>
     <collision>
-      <origin rpy="0.000000 0.000000 0.000000" xyz="-0.027566 -0.000058 -0.009755"/>
-      <geometry>
-        <box size="0.055131 0.089714 0.044510"/>
+      <origin rpy="0.000000 0.000000 0.000000" xyz="-0.027525 -0.000058 -0.010207"/>
+      <geometry>
+        <box size="0.055050 0.089714 0.045413"/>
       </geometry>
     </collision>
@@ -451,5 +451,6 @@
     <parent link="pole_cam_link"/>
     <child link="pole_cam_color_optical_frame"/>
-    <origin rpy="-1.570796 0.000000 -1.570796" xyz="0.000000 0.000000 0.000000"/>
+    <!-- D435 RGB lens: +32.5 mm left of body center, 4.3 mm behind front glass (realsense-ros _d435.urdf.xacro) -->
+    <origin rpy="-1.570796 0.000000 -1.570796" xyz="-0.004300 0.032500 0.000000"/>
   </joint>
   <link name="pole_cam_color_optical_frame"/>
@@ -457,5 +458,6 @@
     <parent link="gripper_cam_link"/>
     <child link="gripper_cam_color_optical_frame"/>
-    <origin rpy="-1.570796 0.000000 -1.570796" xyz="0.000000 0.000000 0.000000"/>
+    <!-- D435 RGB lens: +32.5 mm left of body center, 4.3 mm behind front glass (realsense-ros _d435.urdf.xacro) -->
+    <origin rpy="-1.570796 0.000000 -1.570796" xyz="-0.004300 0.032500 0.000000"/>
   </joint>
   <link name="gripper_cam_color_optical_frame"/>
@@ -466,4 +468,77 @@
     <origin rpy="0 0 0" xyz="-0.064 0 0.068"/>
   </joint>
+  <!-- basket slots: cell floor center, 3 rows (x, pole -> arm) x 4 cols (y, -y -> +y) -->
+  <joint name="basket_slot_0_joint" type="fixed">
+    <parent link="base_link"/>
+    <child link="basket_slot_0"/>
+    <origin rpy="0 0 0" xyz="-0.16984 -0.0975 0.09125"/>
+  </joint>
+  <link name="basket_slot_0"/>
+  <joint name="basket_slot_1_joint" type="fixed">
+    <parent link="base_link"/>
+    <child link="basket_slot_1"/>
+    <origin rpy="0 0 0" xyz="-0.16984 -0.0325 0.09125"/>
+  </joint>
+  <link name="basket_slot_1"/>
+  <joint name="basket_slot_2_joint" type="fixed">
+    <parent link="base_link"/>
+    <child link="basket_slot_2"/>
+    <origin rpy="0 0 0" xyz="-0.16984 0.0325 0.09125"/>
+  </joint>
+  <link name="basket_slot_2"/>
+  <joint name="basket_slot_3_joint" type="fixed">
+    <parent link="base_link"/>
+    <child link="basket_slot_3"/>
+    <origin rpy="0 0 0" xyz="-0.16984 0.0975 0.09125"/>
+  </joint>
+  <link name="basket_slot_3"/>
+  <joint name="basket_slot_4_joint" type="fixed">
+    <parent link="base_link"/>
+    <child link="basket_slot_4"/>
+    <origin rpy="0 0 0" xyz="-0.10484 -0.0975 0.09125"/>
+  </joint>
+  <link name="basket_slot_4"/>
+  <joint name="basket_slot_5_joint" type="fixed">
+    <parent link="base_link"/>
+    <child link="basket_slot_5"/>
+    <origin rpy="0 0 0" xyz="-0.10484 -0.0325 0.09125"/>
+  </joint>
+  <link name="basket_slot_5"/>
+  <joint name="basket_slot_6_joint" type="fixed">
+    <parent link="base_link"/>
+    <child link="basket_slot_6"/>
+    <origin rpy="0 0 0" xyz="-0.10484 0.0325 0.09125"/>
+  </joint>
+  <link name="basket_slot_6"/>
+  <joint name="basket_slot_7_joint" type="fixed">
+    <parent link="base_link"/>
+    <child link="basket_slot_7"/>
+    <origin rpy="0 0 0" xyz="-0.10484 0.0975 0.09125"/>
+  </joint>
+  <link name="basket_slot_7"/>
+  <joint name="basket_slot_8_joint" type="fixed">
+    <parent link="base_link"/>
+    <child link="basket_slot_8"/>
+    <origin rpy="0 0 0" xyz="-0.03984 -0.0975 0.09125"/>
+  </joint>
+  <link name="basket_slot_8"/>
+  <joint name="basket_slot_9_joint" type="fixed">
+    <parent link="base_link"/>
+    <child link="basket_slot_9"/>
+    <origin rpy="0 0 0" xyz="-0.03984 -0.0325 0.09125"/>
+  </joint>
+  <link name="basket_slot_9"/>
+  <joint name="basket_slot_10_joint" type="fixed">
+    <parent link="base_link"/>
+    <child link="basket_slot_10"/>
+    <origin rpy="0 0 0" xyz="-0.03984 0.0325 0.09125"/>
+  </joint>
+  <link name="basket_slot_10"/>
+  <joint name="basket_slot_11_joint" type="fixed">
+    <parent link="base_link"/>
+    <child link="basket_slot_11"/>
+    <origin rpy="0 0 0" xyz="-0.03984 0.0975 0.09125"/>
+  </joint>
+  <link name="basket_slot_11"/>
   <!-- ================= ros2_control ================= -->
   <ros2_control name="BeebotSystem" type="system">
