Commit message: feat: add front caster to usd,urdf

File: lv2_module6/urdf/beebot_mesh/beebot.urdf (robot description, URDF)
Before this commit: robot beebot, 30 links, 29 joints
Links:
- link base_link: geometry collision box size=0.020000 0.020000 0.035350; collision box size=0.020000 0.020000 0.331100
Joints:
- joint front_pole_cam_joint: origin xyz=-0.137869 0.000185 0.434932 rpy=0.000000 0.314159 0.000000 -> xyz=-0.137869 0.000185 0.417108 rpy=0.000000 0.314159 0.000000

File: lv2_module6/urdf/beebot_mesh/urdf.xacro (robot description, xacro)
@@ -28,7 +28,7 @@
   <link name="base_link">
     <inertial>
-      <origin rpy="0 0 0" xyz="-0.085631 -0.000202 0.080552"/>
+      <origin rpy="0 0 0" xyz="-0.085426 -0.000171 0.080461"/>
       <mass value="2.400600"/>
-      <inertia ixx="2.8115e-02" ixy="-1.1729e-05" ixz="6.3963e-03" iyy="3.2571e-02" iyz="-7.6014e-06" izz="2.7719e-02"/>
+      <inertia ixx="2.8130e-02" ixy="-2.1613e-05" ixz="6.4439e-03" iyy="3.2644e-02" iyz="-1.4858e-06" izz="2.7766e-02"/>
     </inertial>
     <visual>
@@ -76,4 +76,18 @@
     <collision>
       <origin rpy="0 0 0" xyz="-0.177000 -0.064000 -0.005237"/>
+      <geometry>
+        <sphere radius="0.004763"/>
+      </geometry>
+    </collision>
+    <!-- front caster (v01) -->
+    <collision>
+      <origin rpy="0 0 0" xyz="0.049600 0.064000 -0.005237"/>
+      <geometry>
+        <sphere radius="0.004763"/>
+      </geometry>
+    </collision>
+    <!-- front caster (v01) -->
+    <collision>
+      <origin rpy="0 0 0" xyz="0.049600 -0.064000 -0.005237"/>
       <geometry>
         <sphere radius="0.004763"/>
@@ -190,5 +204,5 @@
     <parent link="base_link"/>
     <child link="front_pole_cam_link"/>
-    <origin rpy="0.000000 0.314159 0.000000" xyz="-0.137869 0.000185 0.434932"/>
+    <origin rpy="0.000000 0.314159 0.000000" xyz="-0.137869 0.000185 0.417108"/>
   </joint>
   <link name="front_pole_cam_link">

File: lv2_module6/urdf/default/urdf.xacro (robot description, xacro)
@@ -28,7 +28,7 @@
   <link name="base_link">
     <inertial>
-      <origin rpy="0 0 0" xyz="-0.085631 -0.000202 0.080552"/>
+      <origin rpy="0 0 0" xyz="-0.085426 -0.000171 0.080461"/>
       <mass value="2.400600"/>
-      <inertia ixx="2.8115e-02" ixy="-1.1729e-05" ixz="6.3963e-03" iyy="3.2571e-02" iyz="-7.6014e-06" izz="2.7719e-02"/>
+      <inertia ixx="2.8130e-02" ixy="-2.1613e-05" ixz="6.4439e-03" iyy="3.2644e-02" iyz="-1.4858e-06" izz="2.7766e-02"/>
     </inertial>
     <visual>
@@ -76,4 +76,18 @@
     <collision>
       <origin rpy="0 0 0" xyz="-0.177000 -0.064000 -0.005237"/>
+      <geometry>
+        <sphere radius="0.004763"/>
+      </geometry>
+    </collision>
+    <!-- front caster (v01) -->
+    <collision>
+      <origin rpy="0 0 0" xyz="0.049600 0.064000 -0.005237"/>
+      <geometry>
+        <sphere radius="0.004763"/>
+      </geometry>
+    </collision>
+    <!-- front caster (v01) -->
+    <collision>
+      <origin rpy="0 0 0" xyz="0.049600 -0.064000 -0.005237"/>
       <geometry>
         <sphere radius="0.004763"/>
@@ -190,5 +204,5 @@
     <parent link="base_link"/>
     <child link="front_pole_cam_link"/>
-    <origin rpy="0.000000 0.314159 0.000000" xyz="-0.137869 0.000185 0.434932"/>
+    <origin rpy="0.000000 0.314159 0.000000" xyz="-0.137869 0.000185 0.417108"/>
   </joint>
   <link name="front_pole_cam_link">

Commit message: feat: edit pole_front_cam

File: lv2_module6/urdf/beebot_mesh/beebot.urdf (robot description, URDF)
Before this commit: robot beebot, 30 links, 29 joints
Links:
- removed link front_pole_cam_color_optical_frame
- removed link front_pole_cam_link
- added link pole_front_cam_color_optical_frame
- added link pole_front_cam_link, mass 0.072000; collision box size=0.025050 0.089714 0.025000; visual mesh filename=meshes/camera_rear_link.stl scale=0.001 0.001 0.001
Joints:
- removed joint front_pole_cam_joint
- removed joint front_pole_cam_optical_joint
- added joint pole_front_cam_joint: type fixed, parent base_link, child pole_front_cam_link, origin xyz=-0.137869 0.000185 0.417108 rpy=0.000000 0.314159 0.000000
- added joint pole_front_cam_optical_joint: type fixed, parent pole_front_cam_link, child pole_front_cam_color_optical_frame, origin xyz=-0.004300 0.032500 0.000000 rpy=-1.570796 0.000000 -1.570796

File: lv2_module6/urdf/beebot_mesh/urdf.xacro (robot description, xacro)
@@ -3,5 +3,5 @@
   beebot — 실측 CAD(bee.urdf, SolidWorks 내보내기)에서 만든 모델. bee.urdf를 새로 받으면 이 파일을 다시 만든다:
     · 메시 경로: meshes/x.stl → meshes/x.stl
-    · 이름 맞춤(제어·시뮬레이터가 쓰는 이름): camera_rear → front_pole_cam, camera_wrist → gripper_cam,
+    · 이름 맞춤(제어·시뮬레이터가 쓰는 이름): camera_rear → pole_front_cam, camera_wrist → gripper_cam,
       gripper_joint → gripper_left_joint, gripper_mimic_joint → gripper_right_joint, tcp → end_effector
     · 추가: imu_link · <ros2_control> 블록(BeebotSystemHardware) · xacro 인자
@@ -201,10 +201,10 @@
     </collision>
   </link>
-  <joint name="front_pole_cam_joint" type="fixed">
-    <parent link="base_link"/>
-    <child link="front_pole_cam_link"/>
+  <joint name="pole_front_cam_joint" type="fixed">
+    <parent link="base_link"/>
+    <child link="pole_front_cam_link"/>
     <origin rpy="0.000000 0.314159 0.000000" xyz="-0.137869 0.000185 0.417108"/>
   </joint>
-  <link name="front_pole_cam_link">
+  <link name="pole_front_cam_link">
     <inertial>
       <origin rpy="0 0 0" xyz="-0.013393 0.001408 -0.000023"/>
@@ -462,11 +462,11 @@
   </joint>
   <link name="end_effector_link"/>
-  <joint name="front_pole_cam_optical_joint" type="fixed">
-    <parent link="front_pole_cam_link"/>
-    <child link="front_pole_cam_color_optical_frame"/>
+  <joint name="pole_front_cam_optical_joint" type="fixed">
+    <parent link="pole_front_cam_link"/>
+    <child link="pole_front_cam_color_optical_frame"/>
     <!-- D435 RGB lens: +32.5 mm left of body center, 4.3 mm behind front glass (realsense-ros _d435.urdf.xacro) -->
     <origin rpy="-1.570796 0.000000 -1.570796" xyz="-0.004300 0.032500 0.000000"/>
   </joint>
-  <link name="front_pole_cam_color_optical_frame"/>
+  <link name="pole_front_cam_color_optical_frame"/>
   <joint name="gripper_cam_optical_joint" type="fixed">
     <parent link="gripper_cam_link"/>

File: lv2_module6/urdf/beebot_normal/urdf.xacro (robot description, xacro)
@@ -8,5 +8,5 @@
     - 매니퓰레이터: 상판 위 OpenMANIPULATOR-X + 손목 roll — 구동 관절 6개
         joint1 yaw · joint2~4 pitch (OM-X) · joint5 손목 roll (추가) · gripper_left_joint (평행 그리퍼)
-    - 선가이드 폴: 차체 위 뒤쪽 끝, 전원선이 위에서 내려온다. front_pole_cam은 이 폴 위에 전방 하향으로 단다 (가정)
+    - 선가이드 폴: 차체 위 뒤쪽 끝, 전원선이 위에서 내려온다. pole_front_cam은 이 폴 위에 전방 하향으로 단다 (가정)
     - gripper_cam: 그리퍼 몸체(gripper_link) 위에 얹은 RealSense
   xacro 인자:
@@ -189,5 +189,5 @@
     </joint>
   </xacro:macro>
-  <xacro:camera name="front_pole_cam" parent="base_link">
+  <xacro:camera name="pole_front_cam" parent="base_link">
     <origin xyz="${pole_x + 0.020} 0 ${body_top + pole_h}" rpy="0 0.6 0"/>   <!-- 폴 꼭대기 앞, 전방 하향 약 34° -->
   </xacro:camera>

File: lv2_module6/urdf/beebot_slam/urdf.xacro (robot description, xacro)
@@ -3,5 +3,5 @@
   beebot (SLAM 전용) — 지도 스캔할 때 쓰는 모델: 팔·그리퍼·gripper_cam을 떼고, 폴 위 카메라를 앞뒤 두 대로 (더미 치수)
     beebot_normal/urdf.xacro 에서: 매니퓰레이터(arm_base_link ~ finger·end_effector · gripper_cam)와 ros2_control 팔 관절 6개 삭제,
-    폴 꼭대기 반대편(뒤)에 pole_rear_cam 추가 — front_pole_cam은 앞 아래, pole_rear_cam은 뒤 아래를 같은 각도(34°)로 본다.
+    폴 꼭대기 반대편(뒤)에 pole_rear_cam 추가 — pole_front_cam은 앞 아래, pole_rear_cam은 뒤 아래를 같은 각도(34°)로 본다.
     남은 링크·관절 이름은 beebot_mesh · beebot_normal과 같다 (pole_rear_cam만 이 모델에 새로)
   설계: documents/ros2-design/07-tf.md (TF 트리), 08-ctrl.md (ros2_control)
@@ -10,5 +10,5 @@
     - 상판(deck): 차체 위 앞쪽 절반만 덮는 판넬, 스탠드오프 0.05m 위
     - 매니퓰레이터: 없음 (SLAM 전용 — 상판은 그대로)
-    - 선가이드 폴: 차체 위 뒤쪽 끝, 전원선이 위에서 내려온다. 폴 꼭대기 앞쪽에 front_pole_cam(전방 하향) · 뒤쪽에 pole_rear_cam(후방 하향)
+    - 선가이드 폴: 차체 위 뒤쪽 끝, 전원선이 위에서 내려온다. 폴 꼭대기 앞쪽에 pole_front_cam(전방 하향) · 뒤쪽에 pole_rear_cam(후방 하향)
   xacro 인자:
     mock_hardware (false)  true면 control/BeebotSystemHardware가 실기 대신 명령을 그대로 상태로 되돌려 줌 (테스트베드)
@@ -190,5 +190,5 @@
     </joint>
   </xacro:macro>
-  <xacro:camera name="front_pole_cam" parent="base_link">
+  <xacro:camera name="pole_front_cam" parent="base_link">
     <origin xyz="${pole_x + 0.020} 0 ${body_top + pole_h}" rpy="0 0.6 0"/>   <!-- 폴 꼭대기 앞, 전방 하향 약 34° -->
   </xacro:camera>

File: lv2_module6/urdf/default/urdf.xacro (robot description, xacro)
@@ -3,5 +3,5 @@
   beebot — 실측 CAD(bee.urdf, SolidWorks 내보내기)에서 만든 모델. bee.urdf를 새로 받으면 이 파일을 다시 만든다:
     · 메시 경로: meshes/x.stl → meshes/x.stl
-    · 이름 맞춤(제어·시뮬레이터가 쓰는 이름): camera_rear → front_pole_cam, camera_wrist → gripper_cam,
+    · 이름 맞춤(제어·시뮬레이터가 쓰는 이름): camera_rear → pole_front_cam, camera_wrist → gripper_cam,
       gripper_joint → gripper_left_joint, gripper_mimic_joint → gripper_right_joint, tcp → end_effector
     · 추가: imu_link · <ros2_control> 블록(BeebotSystemHardware) · xacro 인자
@@ -201,10 +201,10 @@
     </collision>
   </link>
-  <joint name="front_pole_cam_joint" type="fixed">
-    <parent link="base_link"/>
-    <child link="front_pole_cam_link"/>
+  <joint name="pole_front_cam_joint" type="fixed">
+    <parent link="base_link"/>
+    <child link="pole_front_cam_link"/>
     <origin rpy="0.000000 0.314159 0.000000" xyz="-0.137869 0.000185 0.417108"/>
   </joint>
-  <link name="front_pole_cam_link">
+  <link name="pole_front_cam_link">
     <inertial>
       <origin rpy="0 0 0" xyz="-0.013393 0.001408 -0.000023"/>
@@ -462,11 +462,11 @@
   </joint>
   <link name="end_effector_link"/>
-  <joint name="front_pole_cam_optical_joint" type="fixed">
-    <parent link="front_pole_cam_link"/>
-    <child link="front_pole_cam_color_optical_frame"/>
+  <joint name="pole_front_cam_optical_joint" type="fixed">
+    <parent link="pole_front_cam_link"/>
+    <child link="pole_front_cam_color_optical_frame"/>
     <!-- D435 RGB lens: +32.5 mm left of body center, 4.3 mm behind front glass (realsense-ros _d435.urdf.xacro) -->
     <origin rpy="-1.570796 0.000000 -1.570796" xyz="-0.004300 0.032500 0.000000"/>
   </joint>
-  <link name="front_pole_cam_color_optical_frame"/>
+  <link name="pole_front_cam_color_optical_frame"/>
   <joint name="gripper_cam_optical_joint" type="fixed">
     <parent link="gripper_cam_link"/>
@@ -627,5 +627,5 @@
   <!-- Gazebo (gz-sim): RGBD 카메라 2대. 센서는 optical 프레임 링크에 identity로 — 렌즈가 보는 방향 = optical +Z.
        방향이 뒤집혀 보이면 sensor 안 <pose>에 rpy를 얹어 맞춘다 (URDF optical joint와 같은 값부터). -->
-  <gazebo reference="front_pole_cam_color_optical_frame">
+  <gazebo reference="pole_front_cam_color_optical_frame">
     <sensor name="pole_rgbd" type="rgbd_camera">
       <always_on>true</always_on>
