Commit message: feat: v00 urdf, usd setup

File: lv2_module6/urdf/beebot_mesh/urdf.xacro (robot description, xacro)
@@ -3,5 +3,5 @@
   beebot — 실측 CAD(bee.urdf, SolidWorks 내보내기)에서 만든 모델. bee.urdf를 새로 받으면 이 파일을 다시 만든다:
     · 메시 경로: meshes/x.stl → meshes/x.stl
-    · 이름 맞춤(제어·시뮬레이터가 쓰는 이름): camera_rear → pole_cam, camera_wrist → gripper_cam,
+    · 이름 맞춤(제어·시뮬레이터가 쓰는 이름): camera_rear → front_pole_cam, camera_wrist → gripper_cam,
       gripper_joint → gripper_left_joint, gripper_mimic_joint → gripper_right_joint, tcp → end_effector
     · 추가: imu_link · <ros2_control> 블록(BeebotSystemHardware) · xacro 인자
@@ -187,10 +187,10 @@
     </collision>
   </link>
-  <joint name="pole_cam_joint" type="fixed">
-    <parent link="base_link"/>
-    <child link="pole_cam_link"/>
-    <origin rpy="0.000000 0.314159 0.000000" xyz="-0.137869 0.000185 0.417108"/>
-  </joint>
-  <link name="pole_cam_link">
+  <joint name="front_pole_cam_joint" type="fixed">
+    <parent link="base_link"/>
+    <child link="front_pole_cam_link"/>
+    <origin rpy="0.000000 0.314159 0.000000" xyz="-0.137869 0.000185 0.434932"/>
+  </joint>
+  <link name="front_pole_cam_link">
     <inertial>
       <origin rpy="0 0 0" xyz="-0.013393 0.001408 -0.000023"/>
@@ -214,5 +214,5 @@
     <parent link="base_link"/>
     <child link="arm_base_link"/>
-    <origin rpy="-0.000000 0.000000 0.000000" xyz="0.051045 -0.000000 0.134795"/>
+    <origin rpy="-0.000000 0.000000 0.000000" xyz="0.047985 -0.00023 0.130175"/>
   </joint>
   <link name="arm_base_link">
@@ -421,11 +421,11 @@
     <parent link="gripper_link"/>
     <child link="gripper_cam_link"/>
-    <origin rpy="2.852763 -1.567096 -1.282111" xyz="0.000504 -0.050245 0.080871"/>
+    <origin rpy="0.003448 -1.260182 1.567371" xyz="0.000273 -0.040325 0.081681"/>
   </joint>
   <link name="gripper_cam_link">
     <inertial>
-      <origin rpy="0 0 0" xyz="-0.018065 0.001229 -0.001118"/>
+      <origin rpy="0 0 0" xyz="-0.017727 0.001229 -0.001059"/>
       <mass value="0.088370"/>
-      <inertia ixx="5.1972e-05" ixy="6.5780e-08" ixz="-2.7719e-06" iyy="1.8951e-05" iyz="-6.0902e-08" izz="6.0643e-05"/>
+      <inertia ixx="5.1824e-05" ixy="8.5769e-08" ixz="-2.1898e-06" iyy="1.7218e-05" iyz="-5.7372e-08" izz="5.9057e-05"/>
     </inertial>
     <visual>
@@ -436,7 +436,7 @@
     </visual>
     <collision>
-      <origin rpy="0.000000 0.000000 0.000000" xyz="-0.027566 -0.000058 -0.009755"/>
-      <geometry>
-        <box size="0.055131 0.089714 0.044510"/>
+      <origin rpy="0.000000 0.000000 0.000000" xyz="-0.027525 -0.000058 -0.010207"/>
+      <geometry>
+        <box size="0.055050 0.089714 0.045413"/>
       </geometry>
     </collision>
@@ -448,14 +448,16 @@
   </joint>
   <link name="end_effector_link"/>
-  <joint name="pole_cam_optical_joint" type="fixed">
-    <parent link="pole_cam_link"/>
-    <child link="pole_cam_color_optical_frame"/>
-    <origin rpy="-1.570796 0.000000 -1.570796" xyz="0.000000 0.000000 0.000000"/>
-  </joint>
-  <link name="pole_cam_color_optical_frame"/>
+  <joint name="front_pole_cam_optical_joint" type="fixed">
+    <parent link="front_pole_cam_link"/>
+    <child link="front_pole_cam_color_optical_frame"/>
+    <!-- D435 RGB lens: +32.5 mm left of body center, 4.3 mm behind front glass (realsense-ros _d435.urdf.xacro) -->
+    <origin rpy="-1.570796 0.000000 -1.570796" xyz="-0.004300 0.032500 0.000000"/>
+  </joint>
+  <link name="front_pole_cam_color_optical_frame"/>
   <joint name="gripper_cam_optical_joint" type="fixed">
     <parent link="gripper_cam_link"/>
     <child link="gripper_cam_color_optical_frame"/>
-    <origin rpy="-1.570796 0.000000 -1.570796" xyz="0.000000 0.000000 0.000000"/>
+    <!-- D435 RGB lens: +32.5 mm left of body center, 4.3 mm behind front glass (realsense-ros _d435.urdf.xacro) -->
+    <origin rpy="-1.570796 0.000000 -1.570796" xyz="-0.004300 0.032500 0.000000"/>
   </joint>
   <link name="gripper_cam_color_optical_frame"/>
@@ -466,4 +468,77 @@
     <origin rpy="0 0 0" xyz="-0.064 0 0.068"/>
   </joint>
+  <!-- basket slots: cell floor center, 3 rows (x, pole -> arm) x 4 cols (y, -y -> +y) -->
+  <joint name="basket_slot_0_joint" type="fixed">
+    <parent link="base_link"/>
+    <child link="basket_slot_0"/>
+    <origin rpy="0 0 0" xyz="-0.16984 -0.0975 0.09125"/>
+  </joint>
+  <link name="basket_slot_0"/>
+  <joint name="basket_slot_1_joint" type="fixed">
+    <parent link="base_link"/>
+    <child link="basket_slot_1"/>
+    <origin rpy="0 0 0" xyz="-0.16984 -0.0325 0.09125"/>
+  </joint>
+  <link name="basket_slot_1"/>
+  <joint name="basket_slot_2_joint" type="fixed">
+    <parent link="base_link"/>
+    <child link="basket_slot_2"/>
+    <origin rpy="0 0 0" xyz="-0.16984 0.0325 0.09125"/>
+  </joint>
+  <link name="basket_slot_2"/>
+  <joint name="basket_slot_3_joint" type="fixed">
+    <parent link="base_link"/>
+    <child link="basket_slot_3"/>
+    <origin rpy="0 0 0" xyz="-0.16984 0.0975 0.09125"/>
+  </joint>
+  <link name="basket_slot_3"/>
+  <joint name="basket_slot_4_joint" type="fixed">
+    <parent link="base_link"/>
+    <child link="basket_slot_4"/>
+    <origin rpy="0 0 0" xyz="-0.10484 -0.0975 0.09125"/>
+  </joint>
+  <link name="basket_slot_4"/>
+  <joint name="basket_slot_5_joint" type="fixed">
+    <parent link="base_link"/>
+    <child link="basket_slot_5"/>
+    <origin rpy="0 0 0" xyz="-0.10484 -0.0325 0.09125"/>
+  </joint>
+  <link name="basket_slot_5"/>
+  <joint name="basket_slot_6_joint" type="fixed">
+    <parent link="base_link"/>
+    <child link="basket_slot_6"/>
+    <origin rpy="0 0 0" xyz="-0.10484 0.0325 0.09125"/>
+  </joint>
+  <link name="basket_slot_6"/>
+  <joint name="basket_slot_7_joint" type="fixed">
+    <parent link="base_link"/>
+    <child link="basket_slot_7"/>
+    <origin rpy="0 0 0" xyz="-0.10484 0.0975 0.09125"/>
+  </joint>
+  <link name="basket_slot_7"/>
+  <joint name="basket_slot_8_joint" type="fixed">
+    <parent link="base_link"/>
+    <child link="basket_slot_8"/>
+    <origin rpy="0 0 0" xyz="-0.03984 -0.0975 0.09125"/>
+  </joint>
+  <link name="basket_slot_8"/>
+  <joint name="basket_slot_9_joint" type="fixed">
+    <parent link="base_link"/>
+    <child link="basket_slot_9"/>
+    <origin rpy="0 0 0" xyz="-0.03984 -0.0325 0.09125"/>
+  </joint>
+  <link name="basket_slot_9"/>
+  <joint name="basket_slot_10_joint" type="fixed">
+    <parent link="base_link"/>
+    <child link="basket_slot_10"/>
+    <origin rpy="0 0 0" xyz="-0.03984 0.0325 0.09125"/>
+  </joint>
+  <link name="basket_slot_10"/>
+  <joint name="basket_slot_11_joint" type="fixed">
+    <parent link="base_link"/>
+    <child link="basket_slot_11"/>
+    <origin rpy="0 0 0" xyz="-0.03984 0.0975 0.09125"/>
+  </joint>
+  <link name="basket_slot_11"/>
   <!-- ================= ros2_control ================= -->
   <ros2_control name="BeebotSystem" type="system">

File: lv2_module6/urdf/beebot_normal/urdf.xacro (robot description, xacro)
@@ -8,5 +8,5 @@
     - 매니퓰레이터: 상판 위 OpenMANIPULATOR-X + 손목 roll — 구동 관절 6개
         joint1 yaw · joint2~4 pitch (OM-X) · joint5 손목 roll (추가) · gripper_left_joint (평행 그리퍼)
-    - 선가이드 폴: 차체 위 뒤쪽 끝, 전원선이 위에서 내려온다. pole_cam은 이 폴 위에 전방 하향으로 단다 (가정)
+    - 선가이드 폴: 차체 위 뒤쪽 끝, 전원선이 위에서 내려온다. front_pole_cam은 이 폴 위에 전방 하향으로 단다 (가정)
     - gripper_cam: 그리퍼 몸체(gripper_link) 위에 얹은 RealSense
   xacro 인자:
@@ -189,5 +189,5 @@
     </joint>
   </xacro:macro>
-  <xacro:camera name="pole_cam" parent="base_link">
+  <xacro:camera name="front_pole_cam" parent="base_link">
     <origin xyz="${pole_x + 0.020} 0 ${body_top + pole_h}" rpy="0 0.6 0"/>   <!-- 폴 꼭대기 앞, 전방 하향 약 34° -->
   </xacro:camera>

File: lv2_module6/urdf/beebot_slam/urdf.xacro (robot description, xacro)
@@ -3,5 +3,5 @@
   beebot (SLAM 전용) — 지도 스캔할 때 쓰는 모델: 팔·그리퍼·gripper_cam을 떼고, 폴 위 카메라를 앞뒤 두 대로 (더미 치수)
     beebot_normal/urdf.xacro 에서: 매니퓰레이터(arm_base_link ~ finger·end_effector · gripper_cam)와 ros2_control 팔 관절 6개 삭제,
-    폴 꼭대기 반대편(뒤)에 pole_rear_cam 추가 — pole_cam은 앞 아래, pole_rear_cam은 뒤 아래를 같은 각도(34°)로 본다.
+    폴 꼭대기 반대편(뒤)에 pole_rear_cam 추가 — front_pole_cam은 앞 아래, pole_rear_cam은 뒤 아래를 같은 각도(34°)로 본다.
     남은 링크·관절 이름은 beebot_mesh · beebot_normal과 같다 (pole_rear_cam만 이 모델에 새로)
   설계: documents/ros2-design/07-tf.md (TF 트리), 08-ctrl.md (ros2_control)
@@ -10,5 +10,5 @@
     - 상판(deck): 차체 위 앞쪽 절반만 덮는 판넬, 스탠드오프 0.05m 위
     - 매니퓰레이터: 없음 (SLAM 전용 — 상판은 그대로)
-    - 선가이드 폴: 차체 위 뒤쪽 끝, 전원선이 위에서 내려온다. 폴 꼭대기 앞쪽에 pole_cam(전방 하향) · 뒤쪽에 pole_rear_cam(후방 하향)
+    - 선가이드 폴: 차체 위 뒤쪽 끝, 전원선이 위에서 내려온다. 폴 꼭대기 앞쪽에 front_pole_cam(전방 하향) · 뒤쪽에 pole_rear_cam(후방 하향)
   xacro 인자:
     mock_hardware (false)  true면 control/BeebotSystemHardware가 실기 대신 명령을 그대로 상태로 되돌려 줌 (테스트베드)
@@ -190,5 +190,5 @@
     </joint>
   </xacro:macro>
-  <xacro:camera name="pole_cam" parent="base_link">
+  <xacro:camera name="front_pole_cam" parent="base_link">
     <origin xyz="${pole_x + 0.020} 0 ${body_top + pole_h}" rpy="0 0.6 0"/>   <!-- 폴 꼭대기 앞, 전방 하향 약 34° -->
   </xacro:camera>

File: lv2_module6/urdf/default/urdf.xacro (robot description, xacro)
@@ -3,5 +3,5 @@
   beebot — 실측 CAD(bee.urdf, SolidWorks 내보내기)에서 만든 모델. bee.urdf를 새로 받으면 이 파일을 다시 만든다:
     · 메시 경로: meshes/x.stl → meshes/x.stl
-    · 이름 맞춤(제어·시뮬레이터가 쓰는 이름): camera_rear → pole_cam, camera_wrist → gripper_cam,
+    · 이름 맞춤(제어·시뮬레이터가 쓰는 이름): camera_rear → front_pole_cam, camera_wrist → gripper_cam,
       gripper_joint → gripper_left_joint, gripper_mimic_joint → gripper_right_joint, tcp → end_effector
     · 추가: imu_link · <ros2_control> 블록(BeebotSystemHardware) · xacro 인자
@@ -187,10 +187,10 @@
     </collision>
   </link>
-  <joint name="pole_cam_joint" type="fixed">
-    <parent link="base_link"/>
-    <child link="pole_cam_link"/>
-    <origin rpy="0.000000 0.314159 0.000000" xyz="-0.137869 0.000185 0.417108"/>
-  </joint>
-  <link name="pole_cam_link">
+  <joint name="front_pole_cam_joint" type="fixed">
+    <parent link="base_link"/>
+    <child link="front_pole_cam_link"/>
+    <origin rpy="0.000000 0.314159 0.000000" xyz="-0.137869 0.000185 0.434932"/>
+  </joint>
+  <link name="front_pole_cam_link">
     <inertial>
       <origin rpy="0 0 0" xyz="-0.013393 0.001408 -0.000023"/>
@@ -214,5 +214,5 @@
     <parent link="base_link"/>
     <child link="arm_base_link"/>
-    <origin rpy="-0.000000 0.000000 0.000000" xyz="0.051045 -0.000000 0.134795"/>
+    <origin rpy="-0.000000 0.000000 0.000000" xyz="0.047985 -0.00023 0.130175"/>
   </joint>
   <link name="arm_base_link">
@@ -421,11 +421,11 @@
     <parent link="gripper_link"/>
     <child link="gripper_cam_link"/>
-    <origin rpy="2.852763 -1.567096 -1.282111" xyz="0.000504 -0.050245 0.080871"/>
+    <origin rpy="0.003448 -1.260182 1.567371" xyz="0.000273 -0.040325 0.081681"/>
   </joint>
   <link name="gripper_cam_link">
     <inertial>
-      <origin rpy="0 0 0" xyz="-0.018065 0.001229 -0.001118"/>
+      <origin rpy="0 0 0" xyz="-0.017727 0.001229 -0.001059"/>
       <mass value="0.088370"/>
-      <inertia ixx="5.1972e-05" ixy="6.5780e-08" ixz="-2.7719e-06" iyy="1.8951e-05" iyz="-6.0902e-08" izz="6.0643e-05"/>
+      <inertia ixx="5.1824e-05" ixy="8.5769e-08" ixz="-2.1898e-06" iyy="1.7218e-05" iyz="-5.7372e-08" izz="5.9057e-05"/>
     </inertial>
     <visual>
@@ -436,7 +436,7 @@
     </visual>
     <collision>
-      <origin rpy="0.000000 0.000000 0.000000" xyz="-0.027566 -0.000058 -0.009755"/>
-      <geometry>
-        <box size="0.055131 0.089714 0.044510"/>
+      <origin rpy="0.000000 0.000000 0.000000" xyz="-0.027525 -0.000058 -0.010207"/>
+      <geometry>
+        <box size="0.055050 0.089714 0.045413"/>
       </geometry>
     </collision>
@@ -448,14 +448,16 @@
   </joint>
   <link name="end_effector_link"/>
-  <joint name="pole_cam_optical_joint" type="fixed">
-    <parent link="pole_cam_link"/>
-    <child link="pole_cam_color_optical_frame"/>
-    <origin rpy="-1.570796 0.000000 -1.570796" xyz="0.000000 0.000000 0.000000"/>
-  </joint>
-  <link name="pole_cam_color_optical_frame"/>
+  <joint name="front_pole_cam_optical_joint" type="fixed">
+    <parent link="front_pole_cam_link"/>
+    <child link="front_pole_cam_color_optical_frame"/>
+    <!-- D435 RGB lens: +32.5 mm left of body center, 4.3 mm behind front glass (realsense-ros _d435.urdf.xacro) -->
+    <origin rpy="-1.570796 0.000000 -1.570796" xyz="-0.004300 0.032500 0.000000"/>
+  </joint>
+  <link name="front_pole_cam_color_optical_frame"/>
   <joint name="gripper_cam_optical_joint" type="fixed">
     <parent link="gripper_cam_link"/>
     <child link="gripper_cam_color_optical_frame"/>
-    <origin rpy="-1.570796 0.000000 -1.570796" xyz="0.000000 0.000000 0.000000"/>
+    <!-- D435 RGB lens: +32.5 mm left of body center, 4.3 mm behind front glass (realsense-ros _d435.urdf.xacro) -->
+    <origin rpy="-1.570796 0.000000 -1.570796" xyz="-0.004300 0.032500 0.000000"/>
   </joint>
   <link name="gripper_cam_color_optical_frame"/>
@@ -466,4 +468,77 @@
     <origin rpy="0 0 0" xyz="-0.064 0 0.068"/>
   </joint>
+  <!-- basket slots: cell floor center, 3 rows (x, pole -> arm) x 4 cols (y, -y -> +y) -->
+  <joint name="basket_slot_0_joint" type="fixed">
+    <parent link="base_link"/>
+    <child link="basket_slot_0"/>
+    <origin rpy="0 0 0" xyz="-0.16984 -0.0975 0.09125"/>
+  </joint>
+  <link name="basket_slot_0"/>
+  <joint name="basket_slot_1_joint" type="fixed">
+    <parent link="base_link"/>
+    <child link="basket_slot_1"/>
+    <origin rpy="0 0 0" xyz="-0.16984 -0.0325 0.09125"/>
+  </joint>
+  <link name="basket_slot_1"/>
+  <joint name="basket_slot_2_joint" type="fixed">
+    <parent link="base_link"/>
+    <child link="basket_slot_2"/>
+    <origin rpy="0 0 0" xyz="-0.16984 0.0325 0.09125"/>
+  </joint>
+  <link name="basket_slot_2"/>
+  <joint name="basket_slot_3_joint" type="fixed">
+    <parent link="base_link"/>
+    <child link="basket_slot_3"/>
+    <origin rpy="0 0 0" xyz="-0.16984 0.0975 0.09125"/>
+  </joint>
+  <link name="basket_slot_3"/>
+  <joint name="basket_slot_4_joint" type="fixed">
+    <parent link="base_link"/>
+    <child link="basket_slot_4"/>
+    <origin rpy="0 0 0" xyz="-0.10484 -0.0975 0.09125"/>
+  </joint>
+  <link name="basket_slot_4"/>
+  <joint name="basket_slot_5_joint" type="fixed">
+    <parent link="base_link"/>
+    <child link="basket_slot_5"/>
+    <origin rpy="0 0 0" xyz="-0.10484 -0.0325 0.09125"/>
+  </joint>
+  <link name="basket_slot_5"/>
+  <joint name="basket_slot_6_joint" type="fixed">
+    <parent link="base_link"/>
+    <child link="basket_slot_6"/>
+    <origin rpy="0 0 0" xyz="-0.10484 0.0325 0.09125"/>
+  </joint>
+  <link name="basket_slot_6"/>
+  <joint name="basket_slot_7_joint" type="fixed">
+    <parent link="base_link"/>
+    <child link="basket_slot_7"/>
+    <origin rpy="0 0 0" xyz="-0.10484 0.0975 0.09125"/>
+  </joint>
+  <link name="basket_slot_7"/>
+  <joint name="basket_slot_8_joint" type="fixed">
+    <parent link="base_link"/>
+    <child link="basket_slot_8"/>
+    <origin rpy="0 0 0" xyz="-0.03984 -0.0975 0.09125"/>
+  </joint>
+  <link name="basket_slot_8"/>
+  <joint name="basket_slot_9_joint" type="fixed">
+    <parent link="base_link"/>
+    <child link="basket_slot_9"/>
+    <origin rpy="0 0 0" xyz="-0.03984 -0.0325 0.09125"/>
+  </joint>
+  <link name="basket_slot_9"/>
+  <joint name="basket_slot_10_joint" type="fixed">
+    <parent link="base_link"/>
+    <child link="basket_slot_10"/>
+    <origin rpy="0 0 0" xyz="-0.03984 0.0325 0.09125"/>
+  </joint>
+  <link name="basket_slot_10"/>
+  <joint name="basket_slot_11_joint" type="fixed">
+    <parent link="base_link"/>
+    <child link="basket_slot_11"/>
+    <origin rpy="0 0 0" xyz="-0.03984 0.0975 0.09125"/>
+  </joint>
+  <link name="basket_slot_11"/>
   <!-- ================= ros2_control ================= -->
   <ros2_control name="BeebotSystem" type="system">
@@ -538,5 +613,5 @@
   <!-- Gazebo (gz-sim): RGBD 카메라 2대. 센서는 optical 프레임 링크에 identity로 — 렌즈가 보는 방향 = optical +Z.
        방향이 뒤집혀 보이면 sensor 안 <pose>에 rpy를 얹어 맞춘다 (URDF optical joint와 같은 값부터). -->
-  <gazebo reference="pole_cam_color_optical_frame">
+  <gazebo reference="front_pole_cam_color_optical_frame">
     <sensor name="pole_rgbd" type="rgbd_camera">
       <always_on>true</always_on>
