Commit message: fix: simulator fixed

File: lv2_module6/urdf/beebot_mesh/urdf.xacro (robot description, xacro)
@@ -3,5 +3,5 @@
   beebot — 실측 CAD(bee.urdf, SolidWorks 내보내기)에서 만든 모델. bee.urdf를 새로 받으면 이 파일을 다시 만든다:
     · 메시 경로: meshes/x.stl → meshes/x.stl
-    · 이름 맞춤(제어·시뮬레이터가 쓰는 이름): camera_rear → pole_cam, camera_wrist → gripper_cam,
+    · 이름 맞춤(제어·시뮬레이터가 쓰는 이름): camera_rear → pole_front_cam, camera_wrist → gripper_cam,
       gripper_joint → gripper_left_joint, gripper_mimic_joint → gripper_right_joint, tcp → end_effector
     · 추가: imu_link · <ros2_control> 블록(BeebotSystemHardware) · xacro 인자
@@ -187,10 +187,10 @@
     </collision>
   </link>
-  <joint name="pole_cam_joint" type="fixed">
+  <joint name="pole_front_cam_joint" type="fixed">
     <parent link="base_link"/>
-    <child link="pole_cam_link"/>
+    <child link="pole_front_cam_link"/>
     <origin rpy="0.000000 0.314159 0.000000" xyz="-0.137869 0.000185 0.417108"/>
   </joint>
-  <link name="pole_cam_link">
+  <link name="pole_front_cam_link">
     <inertial>
       <origin rpy="0 0 0" xyz="-0.013393 0.001408 -0.000023"/>
@@ -448,10 +448,10 @@
   </joint>
   <link name="end_effector_link"/>
-  <joint name="pole_cam_optical_joint" type="fixed">
-    <parent link="pole_cam_link"/>
-    <child link="pole_cam_color_optical_frame"/>
+  <joint name="pole_front_cam_optical_joint" type="fixed">
+    <parent link="pole_front_cam_link"/>
+    <child link="pole_front_cam_color_optical_frame"/>
     <origin rpy="-1.570796 0.000000 -1.570796" xyz="0.000000 0.000000 0.000000"/>
   </joint>
-  <link name="pole_cam_color_optical_frame"/>
+  <link name="pole_front_cam_color_optical_frame"/>
   <joint name="gripper_cam_optical_joint" type="fixed">
     <parent link="gripper_cam_link"/>

File: lv2_module6/urdf/beebot_normal/urdf.xacro (robot description, xacro)
@@ -8,5 +8,5 @@
     - 매니퓰레이터: 상판 위 OpenMANIPULATOR-X + 손목 roll — 구동 관절 6개
         joint1 yaw · joint2~4 pitch (OM-X) · joint5 손목 roll (추가) · gripper_left_joint (평행 그리퍼)
-    - 선가이드 폴: 차체 위 뒤쪽 끝, 전원선이 위에서 내려온다. pole_cam은 이 폴 위에 전방 하향으로 단다 (가정)
+    - 선가이드 폴: 차체 위 뒤쪽 끝, 전원선이 위에서 내려온다. pole_front_cam은 이 폴 위에 전방 하향으로 단다 (가정)
     - gripper_cam: 그리퍼 몸체(gripper_link) 위에 얹은 RealSense
   xacro 인자:
@@ -189,5 +189,5 @@
     </joint>
   </xacro:macro>
-  <xacro:camera name="pole_cam" parent="base_link">
+  <xacro:camera name="pole_front_cam" parent="base_link">
     <origin xyz="${pole_x + 0.020} 0 ${body_top + pole_h}" rpy="0 0.6 0"/>   <!-- 폴 꼭대기 앞, 전방 하향 약 34° -->
   </xacro:camera>

File: lv2_module6/urdf/beebot_slam/urdf.xacro (robot description, xacro)
@@ -3,5 +3,5 @@
   beebot (SLAM 전용) — 지도 스캔할 때 쓰는 모델: 팔·그리퍼·gripper_cam을 떼고, 폴 위 카메라를 앞뒤 두 대로 (더미 치수)
     beebot_normal/urdf.xacro 에서: 매니퓰레이터(arm_base_link ~ finger·end_effector · gripper_cam)와 ros2_control 팔 관절 6개 삭제,
-    폴 꼭대기 반대편(뒤)에 pole_rear_cam 추가 — pole_cam은 앞 아래, pole_rear_cam은 뒤 아래를 같은 각도(34°)로 본다.
+    폴 꼭대기 반대편(뒤)에 pole_rear_cam 추가 — pole_front_cam은 앞 아래, pole_rear_cam은 뒤 아래를 같은 각도(34°)로 본다.
     남은 링크·관절 이름은 beebot_mesh · beebot_normal과 같다 (pole_rear_cam만 이 모델에 새로)
   설계: documents/ros2-design/07-tf.md (TF 트리), 08-ctrl.md (ros2_control)
@@ -10,5 +10,5 @@
     - 상판(deck): 차체 위 앞쪽 절반만 덮는 판넬, 스탠드오프 0.05m 위
     - 매니퓰레이터: 없음 (SLAM 전용 — 상판은 그대로)
-    - 선가이드 폴: 차체 위 뒤쪽 끝, 전원선이 위에서 내려온다. 폴 꼭대기 앞쪽에 pole_cam(전방 하향) · 뒤쪽에 pole_rear_cam(후방 하향)
+    - 선가이드 폴: 차체 위 뒤쪽 끝, 전원선이 위에서 내려온다. 폴 꼭대기 앞쪽에 pole_front_cam(전방 하향) · 뒤쪽에 pole_rear_cam(후방 하향)
   xacro 인자:
     mock_hardware (false)  true면 control/BeebotSystemHardware가 실기 대신 명령을 그대로 상태로 되돌려 줌 (테스트베드)
@@ -190,5 +190,5 @@
     </joint>
   </xacro:macro>
-  <xacro:camera name="pole_cam" parent="base_link">
+  <xacro:camera name="pole_front_cam" parent="base_link">
     <origin xyz="${pole_x + 0.020} 0 ${body_top + pole_h}" rpy="0 0.6 0"/>   <!-- 폴 꼭대기 앞, 전방 하향 약 34° -->
   </xacro:camera>

File: lv2_module6/urdf/default/urdf.xacro (robot description, xacro)
@@ -3,5 +3,5 @@
   beebot — 실측 CAD(bee.urdf, SolidWorks 내보내기)에서 만든 모델. bee.urdf를 새로 받으면 이 파일을 다시 만든다:
     · 메시 경로: meshes/x.stl → meshes/x.stl
-    · 이름 맞춤(제어·시뮬레이터가 쓰는 이름): camera_rear → pole_cam, camera_wrist → gripper_cam,
+    · 이름 맞춤(제어·시뮬레이터가 쓰는 이름): camera_rear → pole_front_cam, camera_wrist → gripper_cam,
       gripper_joint → gripper_left_joint, gripper_mimic_joint → gripper_right_joint, tcp → end_effector
     · 추가: imu_link · <ros2_control> 블록(BeebotSystemHardware) · xacro 인자
@@ -16,4 +16,8 @@
 <!-- generated by make_xacro.py -->
 <robot name="beebot" xmlns:xacro="http://www.ros.org/wiki/xacro">
+  <!-- 링크 색상 (STL에 색이 없어 Gazebo·RViz가 하얗게 나옴) -->
+  <material name="beebot_body"><color rgba="0.25 0.27 0.30 1.0"/></material>
+  <material name="beebot_dark"><color rgba="0.10 0.10 0.12 1.0"/></material>
+  <material name="beebot_arm"><color rgba="0.90 0.45 0.10 1.0"/></material>
   <xacro:arg name="mock_hardware" default="false"/>
   <xacro:arg name="mock_effort" default="0.0"/>
@@ -37,4 +41,5 @@
         <mesh filename="$(arg mesh_uri)/base_link.stl" scale="0.001 0.001 0.001"/>
       </geometry>
+      <material name="beebot_body"/>
     </visual>
     <collision>
@@ -85,4 +90,5 @@
         <mesh filename="$(arg mesh_uri)/storage_collision/storage_0.stl" scale="0.001 0.001 0.001"/>
       </geometry>
+      <material name="beebot_body"/>
     </collision>
     <collision name="storage_collision_1">
@@ -91,4 +97,5 @@
         <mesh filename="$(arg mesh_uri)/storage_collision/storage_1.stl" scale="0.001 0.001 0.001"/>
       </geometry>
+      <material name="beebot_body"/>
     </collision>
     <collision name="storage_collision_2">
@@ -97,4 +104,5 @@
         <mesh filename="$(arg mesh_uri)/storage_collision/storage_2.stl" scale="0.001 0.001 0.001"/>
       </geometry>
+      <material name="beebot_body"/>
     </collision>
     <collision name="storage_collision_3">
@@ -103,4 +111,5 @@
         <mesh filename="$(arg mesh_uri)/storage_collision/storage_3.stl" scale="0.001 0.001 0.001"/>
       </geometry>
+      <material name="beebot_body"/>
     </collision>
     <collision name="storage_collision_4">
@@ -109,4 +118,5 @@
         <mesh filename="$(arg mesh_uri)/storage_collision/storage_4.stl" scale="0.001 0.001 0.001"/>
       </geometry>
+      <material name="beebot_body"/>
     </collision>
     <collision name="storage_collision_5">
@@ -115,4 +125,5 @@
         <mesh filename="$(arg mesh_uri)/storage_collision/storage_5.stl" scale="0.001 0.001 0.001"/>
       </geometry>
+      <material name="beebot_body"/>
     </collision>
     <collision name="storage_collision_6">
@@ -121,4 +132,5 @@
         <mesh filename="$(arg mesh_uri)/storage_collision/storage_6.stl" scale="0.001 0.001 0.001"/>
       </geometry>
+      <material name="beebot_body"/>
     </collision>
     <collision name="storage_collision_7">
@@ -127,4 +139,5 @@
         <mesh filename="$(arg mesh_uri)/storage_collision/storage_7.stl" scale="0.001 0.001 0.001"/>
       </geometry>
+      <material name="beebot_body"/>
     </collision>
     <collision name="storage_collision_8">
@@ -133,4 +146,5 @@
         <mesh filename="$(arg mesh_uri)/storage_collision/storage_8.stl" scale="0.001 0.001 0.001"/>
       </geometry>
+      <material name="beebot_body"/>
     </collision>
   </link>
@@ -153,4 +167,5 @@
         <mesh filename="$(arg mesh_uri)/wheel_left_link.stl" scale="0.001 0.001 0.001"/>
       </geometry>
+      <material name="beebot_dark"/>
     </visual>
     <collision>
@@ -179,4 +194,5 @@
         <mesh filename="$(arg mesh_uri)/wheel_right_link.stl" scale="0.001 0.001 0.001"/>
       </geometry>
+      <material name="beebot_dark"/>
     </visual>
     <collision>
@@ -187,10 +203,10 @@
     </collision>
   </link>
-  <joint name="pole_cam_joint" type="fixed">
+  <joint name="pole_front_cam_joint" type="fixed">
     <parent link="base_link"/>
-    <child link="pole_cam_link"/>
+    <child link="pole_front_cam_link"/>
     <origin rpy="0.000000 0.314159 0.000000" xyz="-0.137869 0.000185 0.417108"/>
   </joint>
-  <link name="pole_cam_link">
+  <link name="pole_front_cam_link">
     <inertial>
       <origin rpy="0 0 0" xyz="-0.013393 0.001408 -0.000023"/>
@@ -203,4 +219,5 @@
         <mesh filename="$(arg mesh_uri)/camera_rear_link.stl" scale="0.001 0.001 0.001"/>
       </geometry>
+      <material name="beebot_dark"/>
     </visual>
     <collision>
@@ -227,4 +244,5 @@
         <mesh filename="$(arg mesh_uri)/arm_base_1.stl" scale="0.001 0.001 0.001"/>
       </geometry>
+      <material name="beebot_arm"/>
     </visual>
     <collision name="arm_base_link_collision">
@@ -233,4 +251,5 @@
         <mesh filename="$(arg mesh_uri)/arm_base_1.stl" scale="0.001 0.001 0.001"/>
       </geometry>
+      <material name="beebot_arm"/>
     </collision>
   </link>
@@ -246,4 +265,5 @@
         <mesh filename="$(arg mesh_uri)/shoulder_1.stl" scale="0.001 0.001 0.001"/>
       </geometry>
+      <material name="beebot_arm"/>
     </visual>
     <collision name="shoulder_link_collision">
@@ -252,4 +272,5 @@
         <mesh filename="$(arg mesh_uri)/shoulder_1.stl" scale="0.001 0.001 0.001"/>
       </geometry>
+      <material name="beebot_arm"/>
     </collision>
   </link>
@@ -265,4 +286,5 @@
         <mesh filename="$(arg mesh_uri)/link1_1.stl" scale="0.001 0.001 0.001"/>
       </geometry>
+      <material name="beebot_arm"/>
     </visual>
     <collision name="upper_arm_link_collision">
@@ -271,4 +293,5 @@
         <mesh filename="$(arg mesh_uri)/link1_1.stl" scale="0.001 0.001 0.001"/>
       </geometry>
+      <material name="beebot_arm"/>
     </collision>
   </link>
@@ -284,4 +307,5 @@
         <mesh filename="$(arg mesh_uri)/link2_1.stl" scale="0.001 0.001 0.001"/>
       </geometry>
+      <material name="beebot_arm"/>
     </visual>
     <collision name="forearm_link_collision">
@@ -290,4 +314,5 @@
         <mesh filename="$(arg mesh_uri)/link2_1.stl" scale="0.001 0.001 0.001"/>
       </geometry>
+      <material name="beebot_arm"/>
     </collision>
   </link>
@@ -303,4 +328,5 @@
         <mesh filename="$(arg mesh_uri)/wrist_1.stl" scale="0.001 0.001 0.001"/>
       </geometry>
+      <material name="beebot_arm"/>
     </visual>
     <collision name="wrist_link_collision">
@@ -309,4 +335,5 @@
         <mesh filename="$(arg mesh_uri)/wrist_1.stl" scale="0.001 0.001 0.001"/>
       </geometry>
+      <material name="beebot_arm"/>
     </collision>
   </link>
@@ -322,4 +349,5 @@
         <mesh filename="$(arg mesh_uri)/gripper_body_1.stl" scale="0.001 0.001 0.001"/>
       </geometry>
+      <material name="beebot_dark"/>
     </visual>
     <collision name="gripper_link_collision">
@@ -328,4 +356,5 @@
         <mesh filename="$(arg mesh_uri)/gripper_body_1.stl" scale="0.001 0.001 0.001"/>
       </geometry>
+      <material name="beebot_dark"/>
     </collision>
   </link>
@@ -341,4 +370,5 @@
         <mesh filename="$(arg mesh_uri)/finger_R_1.stl" scale="0.001 0.001 0.001"/>
       </geometry>
+      <material name="beebot_dark"/>
     </visual>
     <collision name="finger_left_link_collision">
@@ -347,4 +377,5 @@
         <mesh filename="$(arg mesh_uri)/finger_R_1.stl" scale="0.001 0.001 0.001"/>
       </geometry>
+      <material name="beebot_dark"/>
     </collision>
   </link>
@@ -360,4 +391,5 @@
         <mesh filename="$(arg mesh_uri)/finger_L_1.stl" scale="0.001 0.001 0.001"/>
       </geometry>
+      <material name="beebot_dark"/>
     </visual>
     <collision name="finger_right_link_collision">
@@ -366,4 +398,5 @@
         <mesh filename="$(arg mesh_uri)/finger_L_1.stl" scale="0.001 0.001 0.001"/>
       </geometry>
+      <material name="beebot_dark"/>
     </collision>
   </link>
@@ -434,4 +467,5 @@
         <mesh filename="$(arg mesh_uri)/camera_wrist_link.stl" scale="0.001 0.001 0.001"/>
       </geometry>
+      <material name="beebot_dark"/>
     </visual>
     <collision>
@@ -448,10 +482,10 @@
   </joint>
   <link name="end_effector_link"/>
-  <joint name="pole_cam_optical_joint" type="fixed">
-    <parent link="pole_cam_link"/>
-    <child link="pole_cam_color_optical_frame"/>
+  <joint name="pole_front_cam_optical_joint" type="fixed">
+    <parent link="pole_front_cam_link"/>
+    <child link="pole_front_cam_color_optical_frame"/>
     <origin rpy="-1.570796 0.000000 -1.570796" xyz="0.000000 0.000000 0.000000"/>
   </joint>
-  <link name="pole_cam_color_optical_frame"/>
+  <link name="pole_front_cam_color_optical_frame"/>
   <joint name="gripper_cam_optical_joint" type="fixed">
     <parent link="gripper_cam_link"/>
@@ -536,20 +570,25 @@
     </sensor>
   </ros2_control>
-  <!-- Gazebo (gz-sim): RGBD 카메라 2대. 센서는 optical 프레임 링크에 identity로 — 렌즈가 보는 방향 = optical +Z.
-       방향이 뒤집혀 보이면 sensor 안 <pose>에 rpy를 얹어 맞춘다 (URDF optical joint와 같은 값부터). -->
-  <gazebo reference="pole_cam_color_optical_frame">
+  <!-- Gazebo (gz-sim): RGBD 카메라 2대.
+       gz 카메라는 센서 프레임의 +X를 본다 → 링크에 identity로 붙여야 정면.
+       (optical 프레임 회전을 센서 pose에 넣으면 카메라가 오른쪽/-Y를 봄) -->
+  <gazebo reference="pole_front_cam_link">
     <sensor name="pole_rgbd" type="rgbd_camera">
+      <pose>0 0 0 0 0 0</pose>
       <always_on>true</always_on>
-      <update_rate>30</update_rate>
-      <topic>pole_cam/rgbd</topic>
+      <!-- RealSense D435 운용 모드: 640×360 @ 15 Hz (원본 640×480 @ 30 Hz보다
+           RGB/depth/point cloud 대역폭을 줄인다). -->
+      <update_rate>15</update_rate>
+      <topic>pole_front_cam/rgbd</topic>
       <camera>
         <horizontal_fov>1.204</horizontal_fov>
-        <image><width>640</width><height>480</height><format>R8G8B8</format></image>
+        <image><width>640</width><height>360</height><format>R8G8B8</format></image>
         <clip><near>0.1</near><far>10.0</far></clip>
       </camera>
     </sensor>
   </gazebo>
-  <gazebo reference="gripper_cam_color_optical_frame">
+  <gazebo reference="gripper_cam_link">
     <sensor name="gripper_rgbd" type="rgbd_camera">
+      <pose>0 0 0 0 0 0</pose>
       <always_on>true</always_on>
       <update_rate>15</update_rate>
@@ -557,7 +596,15 @@
       <camera>
         <horizontal_fov>1.204</horizontal_fov>
-        <image><width>640</width><height>480</height><format>R8G8B8</format></image>
+        <image><width>640</width><height>360</height><format>R8G8B8</format></image>
         <clip><near>0.1</near><far>10.0</far></clip>
       </camera>
+    </sensor>
+  </gazebo>
+  <!-- IMU (base_link, 100Hz) — RealSense 내장 IMU 대응. /imu(하드웨어·목mock)와 안 겹치게 /imu_gz로 나감 -->
+  <gazebo reference="base_link">
+    <sensor name="imu" type="imu">
+      <always_on>true</always_on>
+      <update_rate>100</update_rate>
+      <topic>imu</topic>
     </sensor>
   </gazebo>
@@ -580,15 +627,26 @@
       <publish_odom_tf>false</publish_odom_tf>
     </plugin>
-    <plugin filename="libgz-sim-joint-position-controller-system.so" name="gz::sim::systems::JointPositionController">
-      <joint_name>joint1</joint_name>
-      <joint_name>joint2</joint_name>
-      <joint_name>joint3</joint_name>
-      <joint_name>joint4</joint_name>
-      <joint_name>joint5</joint_name>
-      <joint_name>gripper_left_joint</joint_name>
-      <joint_name>gripper_right_joint</joint_name>
-      <initial_position>0</initial_position>
-      <p_gain>10</p_gain>
-    </plugin>
+    <!-- JointPositionController는 플러그인 1개 = 관절 1개만 제어한다.
+         한 플러그인에 joint_name을 여러 개 넣으면 첫 개만 잡혀서 나머지 팔이 중력에 접힌다. -->
+    <xacro:macro name="gz_jpc" params="joint effort:=4.1">
+      <plugin filename="libgz-sim-joint-position-controller-system.so" name="gz::sim::systems::JointPositionController">
+        <joint_name>${joint}</joint_name>
+        <initial_position>0</initial_position>
+        <p_gain>50</p_gain>
+        <i_gain>5</i_gain>
+        <d_gain>1</d_gain>
+        <i_max>${effort}</i_max>
+        <i_min>-${effort}</i_min>
+        <cmd_max>${effort}</cmd_max>
+        <cmd_min>-${effort}</cmd_min>
+      </plugin>
+    </xacro:macro>
+    <xacro:gz_jpc joint="joint1"/>
+    <xacro:gz_jpc joint="joint2"/>
+    <xacro:gz_jpc joint="joint3"/>
+    <xacro:gz_jpc joint="joint4"/>
+    <xacro:gz_jpc joint="joint5"/>
+    <xacro:gz_jpc joint="gripper_left_joint" effort="20"/>
+    <xacro:gz_jpc joint="gripper_right_joint" effort="20"/>
   </gazebo>
 </robot>

Commit message: feature: jetson nano parameter if

File: lv2_module6/urdf/beebot_mesh/urdf.xacro (robot description, xacro)
@@ -469,4 +469,12 @@
   </joint>
   <link name="pole_front_cam_color_optical_frame"/>
+  <joint name="pole_front_cam_depth_optical_joint" type="fixed">
+    <parent link="pole_front_cam_link"/>
+    <child link="pole_front_cam_depth_optical_frame"/>
+    <!-- RealSense point cloud is published in the depth optical frame. publish_tf=false라
+         (publish_tf는 URDF와 중복 방지용) 이 고정 프레임을 URDF가 제공해야 한다. -->
+    <origin rpy="-1.570796 0.000000 -1.570796" xyz="0.000000 0.000000 0.000000"/>
+  </joint>
+  <link name="pole_front_cam_depth_optical_frame"/>
   <joint name="gripper_cam_optical_joint" type="fixed">
     <parent link="gripper_cam_link"/>
@@ -475,4 +483,10 @@
   </joint>
   <link name="gripper_cam_color_optical_frame"/>
+  <joint name="gripper_cam_depth_optical_joint" type="fixed">
+    <parent link="gripper_cam_link"/>
+    <child link="gripper_cam_depth_optical_frame"/>
+    <origin rpy="-1.570796 0.000000 -1.570796" xyz="0.000000 0.000000 0.000000"/>
+  </joint>
+  <link name="gripper_cam_depth_optical_frame"/>
   <link name="imu_link"/>
   <joint name="imu_joint" type="fixed">

File: lv2_module6/urdf/default/urdf.xacro (robot description, xacro)
@@ -503,4 +503,12 @@
   </joint>
   <link name="pole_front_cam_color_optical_frame"/>
+  <joint name="pole_front_cam_depth_optical_joint" type="fixed">
+    <parent link="pole_front_cam_link"/>
+    <child link="pole_front_cam_depth_optical_frame"/>
+    <!-- RealSense point cloud is published in the depth optical frame. publish_tf=false라
+         (publish_tf는 URDF와 중복 방지용) 이 고정 프레임을 URDF가 제공해야 한다. -->
+    <origin rpy="-1.570796 0.000000 -1.570796" xyz="0.000000 0.000000 0.000000"/>
+  </joint>
+  <link name="pole_front_cam_depth_optical_frame"/>
   <joint name="gripper_cam_optical_joint" type="fixed">
     <parent link="gripper_cam_link"/>
@@ -509,4 +517,10 @@
   </joint>
   <link name="gripper_cam_color_optical_frame"/>
+  <joint name="gripper_cam_depth_optical_joint" type="fixed">
+    <parent link="gripper_cam_link"/>
+    <child link="gripper_cam_depth_optical_frame"/>
+    <origin rpy="-1.570796 0.000000 -1.570796" xyz="0.000000 0.000000 0.000000"/>
+  </joint>
+  <link name="gripper_cam_depth_optical_frame"/>
   <link name="imu_link"/>
   <joint name="imu_joint" type="fixed">

Commit message: fix: manipulator offset and SBC

File: lv2_module6/urdf/beebot_mesh/urdf.xacro (robot description, xacro)
@@ -515,4 +515,5 @@
     </joint>
     <joint name="joint1">
+      <param name="offset">0.0</param>  <!-- [rad] 영점 오프셋: 서보 값 = 관절값 + offset (실측) -->
       <command_interface name="position"/>
       <state_interface name="position"/>
@@ -521,4 +522,5 @@
     </joint>
     <joint name="joint2">
+      <param name="offset">0.0</param>  <!-- [rad] 영점 오프셋: 서보 값 = 관절값 + offset (실측) -->
       <command_interface name="position"/>
       <state_interface name="position"/>
@@ -527,4 +529,5 @@
     </joint>
     <joint name="joint3">
+      <param name="offset">0.0</param>  <!-- [rad] 영점 오프셋: 서보 값 = 관절값 + offset (실측) -->
       <command_interface name="position"/>
       <state_interface name="position"/>
@@ -533,4 +536,5 @@
     </joint>
     <joint name="joint4">
+      <param name="offset">0.0</param>  <!-- [rad] 영점 오프셋: 서보 값 = 관절값 + offset (실측) -->
       <command_interface name="position"/>
       <state_interface name="position"/>
@@ -539,4 +543,5 @@
     </joint>
     <joint name="joint5">
+      <param name="offset">0.0</param>  <!-- [rad] 영점 오프셋: 서보 값 = 관절값 + offset (실측) -->
       <command_interface name="position"/>
       <state_interface name="position"/>
@@ -545,4 +550,5 @@
     </joint>
     <joint name="gripper_left_joint">
+      <param name="offset">0.0</param>  <!-- [m] 영점 오프셋: 서보 값 = 관절값 + offset (실측) -->
       <command_interface name="position"/>
       <state_interface name="position"/>

File: lv2_module6/urdf/beebot_normal/urdf.xacro (robot description, xacro)
@@ -290,6 +290,7 @@
     <xacro:wheel_if name="wheel_left_joint"/>
     <xacro:wheel_if name="wheel_right_joint"/>
-    <xacro:macro name="arm_if" params="name">
+    <xacro:macro name="arm_if" params="name offset:=0.0">
       <joint name="${name}">
+        <param name="offset">${offset}</param>  <!-- 영점 오프셋 [rad·그리퍼 m]: 서보 값 = 관절값 + offset (실측) -->
         <command_interface name="position"/>
         <state_interface name="position"/>

File: lv2_module6/urdf/default/urdf.xacro (robot description, xacro)
@@ -549,4 +549,5 @@
     </joint>
     <joint name="joint1">
+      <param name="offset">0.0</param>  <!-- [rad] 영점 오프셋: 서보 값 = 관절값 + offset (실측) -->
       <command_interface name="position"/>
       <state_interface name="position"/>
@@ -555,4 +556,5 @@
     </joint>
     <joint name="joint2">
+      <param name="offset">0.0</param>  <!-- [rad] 영점 오프셋: 서보 값 = 관절값 + offset (실측) -->
       <command_interface name="position"/>
       <state_interface name="position"/>
@@ -561,4 +563,5 @@
     </joint>
     <joint name="joint3">
+      <param name="offset">0.0</param>  <!-- [rad] 영점 오프셋: 서보 값 = 관절값 + offset (실측) -->
       <command_interface name="position"/>
       <state_interface name="position"/>
@@ -567,4 +570,5 @@
     </joint>
     <joint name="joint4">
+      <param name="offset">0.0</param>  <!-- [rad] 영점 오프셋: 서보 값 = 관절값 + offset (실측) -->
       <command_interface name="position"/>
       <state_interface name="position"/>
@@ -573,4 +577,5 @@
     </joint>
     <joint name="joint5">
+      <param name="offset">0.0</param>  <!-- [rad] 영점 오프셋: 서보 값 = 관절값 + offset (실측) -->
       <command_interface name="position"/>
       <state_interface name="position"/>
@@ -579,4 +584,5 @@
     </joint>
     <joint name="gripper_left_joint">
+      <param name="offset">0.0</param>  <!-- [m] 영점 오프셋: 서보 값 = 관절값 + offset (실측) -->
       <command_interface name="position"/>
       <state_interface name="position"/>
